Commit message: change in urdf

File: kridtbot/description/robot.urdf.xacro (robot description, xacro)
@@ -2,4 +2,4 @@
 <robot xmlns:xacro="http://www.ros.org/wiki/xacro"  name="robot">
     <!-- Example link -->
-    <link name="base_link1"></link>
+    <link name="base_link1123"></link>
 </robot>

Commit message: w

File: kridtbot/description/robot.urdf.xacro (robot description, xacro)
@@ -2,4 +2,4 @@
 <robot xmlns:xacro="http://www.ros.org/wiki/xacro"  name="robot">
     <!-- Example link -->
-    <link name="base_link1"></link>
+    <link name="base_link"></link>
 </robot>

Commit message: w

File: kridtbot/description/robot.urdf.xacro (robot description, xacro)
@@ -2,4 +2,4 @@
 <robot xmlns:xacro="http://www.ros.org/wiki/xacro"  name="robot">
     <!-- Example link -->
-    <link name="base_link1123"></link>
+    <link name="base_link1"></link>
 </robot>

Commit message: w

File: kridtbot/description/robot.urdf.xacro (robot description, xacro)
@@ -1,5 +1,4 @@
 <?xml version="1.0"?>
 <robot xmlns:xacro="http://www.ros.org/wiki/xacro"  name="robot">
-    <!-- Example link -->
-    <link name="base_link1"></link>
+    <xacro:include filename="robot_coer.xacro" />
 </robot>

Commit message: fr

File: kridtbot/description/robot.urdf.xacro (robot description, xacro)
@@ -2,4 +2,3 @@
 <robot xmlns:xacro="http://www.ros.org/wiki/xacro"  name="robot">
     <xacro:include filename="robot_core.xacro" />
-    <xacro:include filename="$(find kridtbot)/meshes/base_link.STL" />
 </robot>

File: kridtbot/description/robot_core.xacro (robot description, xacro)
@@ -8,5 +8,5 @@
         rpy="0 0 0" />
       <geometry>
-        <mesh filename="$(find kridtbot)/meshes/base_link.STL" />
+        <mesh filename="package://kridtbot/meshes/base_link.STL" />
       </geometry>
       <material

Commit message: r

File: kridtbot/description/robot.urdf.xacro (robot description, xacro)
@@ -4,4 +4,4 @@
     <xacro:include filename="robot_core.xacro" />
     <!-- Gazebo ros2_control plugins-->
-    <!--<xacro:include filename="gazebo_control.xacro" /> -->
+    <xacro:include filename="gazebo_control.xacro" />
 </robot>

File: kridtbot/description/robot_core.xacro (robot description, xacro)
@@ -71,4 +71,5 @@
     <parent link="diff_link"/>
     <child link="left_diff_link"/>
+    <mimic joint="diff_to_right_diff" multiplyer="-1.0"/>
   </joint>
   <!-- _____________LEFT DIFF LINK____________-->
