Commit message: w

File: kridtbot/description/gazebo_control.xacro (robot description, xacro)
@@ -3,19 +3,16 @@
 <!-- Inspired from: https://www.youtube.com/watch?v=IjFcr5r0nMs&list=PLunhqkrRNRhYAffV8JDiFOatQXuU-NnxT&index=3-->
 <robot xmlns:xacro="http://www.ros.org/wiki/xacro">
-    <!-- Variables -->
-    <xacro:property name="d_wheel" value="$0.0163" /> <!-- [m] from urdf -->
-    <xacro:property name="wheelSeparation" value="$0.068185" /> <!-- [m] from SW -->
     <!-- Gazebo ros2_control plugins-->
     <gazebo>
         <plugin name="gazebo_2w_diff" filename="libgazebo_ros_diff_drive.so">
             <!-- Properties-->
-            <wheelSeparation>wheelSeparation</wheelSeparation>
-            <wheelDiameter>d_wheel</wheelDiameter>
+            <wheelSeparation>0.068185"</wheelSeparation>  <!-- [m] from SW -->
+            <wheelDiameter>0.0163</wheelDiameter> <!-- [m] from urdf -->
             <left_joint>left_rear_lin_to_left_rear_rev</left_joint>
-            <right_joint>right_rear_lin_to_right_rear_rev</right_joint>
+            <right_joint>right_rear_lin_to_right_rear_re</right_joint>
             <!-- Limits -->
-            <max_wheel_torque>100.0</max_wheel_torque> <!-- !!!! CHANGE !!!! -->
-            <max_acceleration>5</max_acceleration> <!-- !!!! CHANGE !!!! -->
-            <!-- Odometry -->
+            <max_wheel_torque>10.0</max_wheel_torque> <!-- !!!! CHANGE !!!! -->
+            <max_acceleration>0.5</max_acceleration> <!-- !!!! CHANGE !!!! -->
+            <!-- Output -->
             <odometry_frame>odom</odometry_frame>
             <robot_base_frame>base_link</robot_base_frame>

Commit message: w

File: kridtbot/description/gazebo_control.xacro (robot description, xacro)
@@ -4,6 +4,6 @@
         <plugin name="gz::sim::systems::DiffDrive" filename="gz-sim-diff-drive-system">
             <!-- Wheel Information -->
-            <left_joint>left_rear_lin_to_left_rear_rev</left_joint>
-            <right_joint>right_rear_lin_to_right_rear_rev</right_joint>
+            <left_joint>left_rear_wheel</left_joint>
+            <right_joint>right_rear_wheel</right_joint>
             <!-- [m] from SW -->
             <wheel_seperation>0.068185</wheel_seperation>
@@ -24,6 +24,6 @@
             name="gz::sim::systems::JointStatePublisher">
             <topic>joint_states</topic>
-            <joint_name>left_rear_lin_to_left_rear_rev</joint_name>
-            <joint_name>right_rear_lin_to_right_rear_rev</joint_name>
+            <joint_name>left_rear_wheel</joint_name>
+            <joint_name>right_rear_wheel</joint_name>
         </plugin>
     </gazebo>

File: kridtbot/description/robot.urdf.xacro (robot description, xacro)
@@ -4,6 +4,6 @@
     <xacro:include filename="robot_core.xacro" />
     <!-- Gazebo ros2_control plugins-->
-    <xacro:include filename="gazebo_control.xacro" />
+    <!--<xacro:include filename="gazebo_control.xacro" />-->
     <!-- ROS2 Control plugins-->
-    <!--<xacro:include filename="ros2_control.xacro" /> -->
+    <xacro:include filename="ros2_control.xacro" />
 </robot>

File: kridtbot/description/robot_core.xacro (robot description, xacro)
@@ -82,5 +82,5 @@
   </gazebo>
   <!-- _____________DIFF TO LEFT DIFF JOINT____________-->
-  <joint name="diff_to_left_diff" type="revolute">
+  <joint name="left_diff" type="revolute"> <!--diff_to_left_diff-->
     <origin xyz="0 0 -0.28" rpy="-3.1416 0 -3.1416"/>
     <axis xyz="0 0 1"/>
@@ -116,5 +116,5 @@
   </gazebo>
   <!-- _____________LEFT DIFF TO LEFT REAR LIN JOINT____________-->
-  <joint name="left_diff_to_left_rear_lin" type="prismatic">
+  <joint name="left_rear_linear" type="prismatic"> <!-- left_diff_to_left_rear_lin -->
     <limit effort="1000.0" lower="0" upper="0.13" velocity="0.5"/>
     <origin xyz="-0.216 -0.0010724 0" rpy="-1.5708 0 0.0049647"/>
@@ -148,5 +148,5 @@
   </gazebo>
 <!-- _____________LEFT REAR LIN TO LEFT REAR REV JOINT____________-->
-  <joint name="left_rear_lin_to_left_rear_rev" type="continuous">
+  <joint name="left_rear_wheel" type="continuous"> <!-- left_rear_lin_to_left_rear_rev -->
     <origin xyz="0.0012158 0 0.2449" rpy="1.5708 0 0"/>
     <axis xyz="0 0 1"/>
@@ -179,5 +179,5 @@
   </gazebo>
     <!-- _____________LEFT DIFF TO LEFT FRONT LIN JOINT____________-->
-  <joint name="left_diff_to_left_front_lin" type="prismatic">
+  <joint name="left_front_linear" type="prismatic"> <!-- left_diff_to_left_front_lin-->
     <limit effort="1000.0" lower="0" upper="0.13" velocity="0.5"/>
     <origin xyz="0.216 0.0010724 0" rpy="-1.5708 0 0.0049647"/>
@@ -211,5 +211,5 @@
   </gazebo>
 <!-- _____________LEFT FRONT LIN TO LEFT FRONT REV JOINT____________-->
-  <joint name="left_front_lin_to_left_front_rev" type="continuous">
+  <joint name="left_front_wheel" type="continuous"> <!-- left_front_lin_to_left_front_rev -->
     <origin xyz="0.0012158 0 0.2449" rpy="1.5708 0 0"/>
     <axis xyz="0 0 1"/>
@@ -239,10 +239,10 @@
     <gazebo reference="left_front_rev_link">
       <material>Gazebo/Orange</material>
-      <mu1 value = "0.001"/>
-      <mu2 value = "0.001"/>
+      <mu1 value = "0.5"/>
+      <mu2 value = "0.5"/>
     </gazebo>
   </link>
     <!-- _____________DIFF TO RIGHT DIFF JOINT____________-->
-    <joint name="diff_to_right_diff" type="revolute">
+    <joint name="right_diff" type="revolute"> <!-- diff_to_right_diff -->
       <origin xyz="0 0 0.28" rpy="0 0 0"/>
       <axis xyz="0 0 1"/>
@@ -250,5 +250,5 @@
       <parent link="diff_link"/>
       <child link="right_diff_link"/>
-      <mimic joint="diff_to_left_diff" multiplier="1"/>
+      <mimic joint="left_diff" multiplier="1"/>
     </joint>
     <!-- _____________RIGHT DIFF LINK____________-->
@@ -279,5 +279,5 @@
     </gazebo>
     <!-- _____________RIGHT DIFF TO RIGHT REAR LIN JOINT____________-->
-    <joint name="right_diff_to_right_rear_lin" type="prismatic">
+    <joint name="right_rear_linear" type="prismatic"> <!-- right_diff_to_right_rear_lin -->
       <limit effort="1000.0" lower="0" upper="0.13" velocity="0.5"/>
       <origin xyz="-0.216 -0.0010724 0" rpy="-1.5708 0 0.0049647"/>
@@ -311,5 +311,5 @@
     </gazebo>
   <!-- _____________RIGHT REAR LIN TO RIGHT REAR REV JOINT____________-->
-    <joint name="right_rear_lin_to_right_rear_rev" type="continuous">
+    <joint name="right_rear_wheel" type="continuous"> <!-- right_rear_lin_to_right_rear_rev -->
       <origin xyz="0.0012158 0 0.2449" rpy="1.5708 0 0"/>
       <axis xyz="0 0 1"/>
@@ -342,5 +342,5 @@
     </gazebo>
       <!-- _____________RIGHT DIFF TO RIGHT FRONT LIN JOINT____________-->
-    <joint name="right_diff_to_right_front_lin" type="prismatic">
+    <joint name="right_front_linear" type="prismatic"> <!-- right_diff_to_right_front_lin -->
       <limit effort="1000.0" lower="0" upper="0.13" velocity="0.5"/>
       <origin xyz="0.216 0.0010724 0" rpy="-1.5708 0 0.0049647"/>
@@ -374,5 +374,5 @@
     </gazebo>
   <!-- _____________RIGHT FRONT LIN TO RIGHT FRONT REV JOINT____________-->
-    <joint name="right_front_lin_to_right_front_rev" type="continuous">
+    <joint name="right_front_wheel" type="continuous"> <!-- right_front_lin_to_right_front_rev -->
       <origin xyz="0.0012158 0 0.2449" rpy="1.5708 0 0"/>
       <axis xyz="0 0 1"/>
@@ -403,6 +403,6 @@
     <gazebo reference="right_front_rev_link">
       <material>Gazebo/Orange</material>
-      <mu1 value = "0.001"/>
-      <mu2 value = "0.001"/>
+      <mu1 value = "0.5"/>
+      <mu2 value = "0.5"/>
     </gazebo>
 </robot>

File: kridtbot/description/ros2_control.xacro (robot description, xacro)
@@ -8,5 +8,5 @@
         </hardware>
         <!-- All continous joints-->
-        <joint name="left_rear_lin_to_left_rear_rev">
+        <joint name="left_rear_wheel">
             <command_interface name="velocity">
                 <param name="min">-10</param>
@@ -21,5 +21,5 @@
             <!--<state_interface name="voltage"></state_interface> --><!-- Not sure if this is needed -->
         </joint>
-        <joint name="right_rear_lin_to_right_rear_rev">
+        <joint name="right_rear_wheel">
             <command_interface name="velocity">
                 <param name="min">-10</param>
@@ -34,5 +34,5 @@
             <!--<state_interface name="voltage"></state_interface> --><!-- Not sure if this is needed -->
         </joint>
-        <joint name="left_front_lin_to_left_front_rev">
+        <joint name="left_front_wheel">
             <command_interface name="velocity">
                 <param name="min">-10</param>
@@ -47,5 +47,5 @@
             <!--<state_interface name="voltage"></state_interface> --><!-- Not sure if this is needed -->
         </joint>
-        <joint name="right_front_lin_to_right_front_rev">
+        <joint name="right_front_wheel">
             <command_interface name="velocity">
                 <param name="min">-10</param>
@@ -64,6 +64,7 @@
     <gazebo>
         <plugin name="gz_ros2_control::GazeboSimROS2ControlPlugin" filename="libgz_ros2_control-system.so">
-            <!--<parameters>$(find kridtbot)/config/my_controllers.yaml </parameters> -->
-            <parameters>filename="file:$(find kridtbot)/config/my_controllers.yaml"</parameters>
+            <parameters>$(find kridtbot)/config/mycontrollers.yaml</parameters>
+            <!--<parameters filename="file:$(find kridtbot)/config/my_controllers.yaml"/> -->
+            <!--<parameters>filename="file:$(find kridtbot)/config/my_controllers.yaml"</parameters> -->
         </plugin>
     </gazebo>
