Commit message: Changes to URDF

File: kridtbot/description/imu_core.xacro (robot description, xacro)
@@ -1,4 +1,7 @@
 <?xml version="1.0"?>
 <robot xmlns:xacro="http://www.ros.org/wiki/xacro">
+  <material name="black">
+    <color rgba="${64/255} ${64/255} ${64/255} 1" />
+  </material>
   <!-- _____________IMU LINK____________-->
   <link name="imu_link">
@@ -18,6 +21,6 @@
     </collision>
     <inertial>
-      <mass value="1.44"/>
-      <inertia ixx="2024193.31e-9" ixy="258.53e-9" ixz="-42.56e-9" iyy="1553917.67e-9" iyz=" 559.93e-9" izz="1298088.14e-9"/>
+      <mass value="0.02302"/>
+      <inertia ixx="3763.33e-9" ixy="0" ixz="0" iyy="6942.61e-9" iyz="0" izz="9041.46e-9"/>
     </inertial>
   </link>
@@ -27,5 +30,5 @@
   <!-- _____________DIFF TO IMU JOINT____________-->
   <joint name="diff_to_imu" type="fixed">
-    <origin xyz="0 0 0" rpy="0 0 0"/>
+    <origin xyz="-0.038 0 0" rpy="1.57079633 0 1.57079633"/>
     <parent link="diff_link"/>
     <child link="imu_link"/>

Commit message: f

File: kridtbot/description/imu_core.xacro (robot description, xacro)
@@ -30,7 +30,10 @@
   <!-- _____________DIFF TO IMU JOINT____________-->
   <joint name="diff_to_imu" type="fixed">
-    <origin xyz="-0.038 0 0" rpy="1.57079633 0 1.57079633"/>
+    <origin xyz="-1.0 0 0" rpy="1.57079633 0 1.57079633"/>
     <parent link="diff_link"/>
     <child link="imu_link"/>
   </joint>
+  <gazebo reference="imu_link">
+    <material>Gazebo/Black</material>
+  </gazebo>
 </robot>

File: kridtbot/description/robot.urdf.xacro (robot description, xacro)
@@ -3,5 +3,4 @@
     <!-- URDF Robot Description-->
     <xacro:include filename="robot_core.xacro" />
-    <!--xacro:include filename="imu_core.xacro"-->
     <!-- Gazebo ros2_control plugins-->
     <!--<xacro:include filename="gazebo_control.xacro" />-->

File: kridtbot/description/robot_core.xacro (robot description, xacro)
@@ -81,4 +81,36 @@
     <material>Gazebo/Orange</material>
   </gazebo>
+  <link name="imu_link">
+    <visual>
+      <origin xyz="0 0 0" rpy="0 0 0"/>
+      <geometry>
+        <mesh filename="file:$(find kridtbot)/meshes/imu_link.STL"/>
+      </geometry>
+      <material name = "black"/>
+    </visual>
+    <collision>
+      <origin xyz="0 0 0" rpy="0 0 0"/>
+      <geometry>
+        <mesh filename="file:$(find kridtbot)/meshes/imu_link.STL"/>
+      </geometry>
+      <material name="mesh_color"/>
+    </collision>
+    <inertial>
+      <mass value="0.02302"/>
+      <inertia ixx="3763.33e-9" ixy="0" ixz="0" iyy="6942.61e-9" iyz="0" izz="9041.46e-9"/>
+    </inertial>
+  </link>
+  <gazebo reference="imu_link">
+    <material>Gazebo/Orange</material>
+  </gazebo>
+  <!-- _____________DIFF TO IMU JOINT____________-->
+  <joint name="diff_to_imu" type="fixed">
+    <origin xyz="-1.0 0 0" rpy="1.57079633 0 1.57079633"/>
+    <parent link="diff_link"/>
+    <child link="imu_link"/>
+  </joint>
+  <gazebo reference="imu_link">
+    <material>Gazebo/Black</material>
+  </gazebo>
   <!-- _____________DIFF TO LEFT DIFF JOINT____________-->
   <joint name="left_diff" type="revolute"> <!--diff_to_left_diff-->
