Commit message: urdf input

File: kridtbot/description/robot_core.xacro (robot description, xacro)
@@ -1,3 +1,656 @@
 <?xml version="1.0"?>
 <robot xmlns:xacro="http://www.ros.org/wiki/xacro">
+    <link
+    name="base_link">
+    <inertial>
+      <origin
+        xyz="-0.00062572 0.0029573 -0.11694"
+        rpy="0 0 0" />
+      <mass
+        value="3.8611" />
+      <inertia
+        ixx="0.1509"
+        ixy="-3.2679E-16"
+        ixz="-3.3043E-17"
+        iyy="0.14248"
+        iyz="-0.0045004"
+        izz="0.19616" />
+    </inertial>
+    <visual>
+      <origin
+        xyz="0 0 0"
+        rpy="0 0 0" />
+      <geometry>
+        <mesh
+          filename="package://KridtBot/meshes/base_link.STL" />
+      </geometry>
+      <material
+        name="">
+        <color
+          rgba="0.98824 0.73725 0.51765 1" />
+      </material>
+    </visual>
+    <collision>
+      <origin
+        xyz="0 0 0"
+        rpy="0 0 0" />
+      <geometry>
+        <mesh
+          filename="package://KridtBot/meshes/base_link.STL" />
+      </geometry>
+    </collision>
+  </link>
+  <link
+    name="diff_link">
+    <inertial>
+      <origin
+        xyz="6.3148E-06 0.0091271 1.2916E-05"
+        rpy="0 0 0" />
+      <mass
+        value="2.9137" />
+      <inertia
+        ixx="0.0037228"
+        ixy="5.5526E-08"
+        ixz="1.4073E-07"
+        iyy="0.0030992"
+        iyz="1.4623E-08"
+        izz="0.0022766" />
+    </inertial>
+    <visual>
+      <origin
+        xyz="0 0 0"
+        rpy="0 0 0" />
+      <geometry>
+        <mesh
+          filename="package://KridtBot/meshes/diff_link.STL" />
+      </geometry>
+      <material
+        name="">
+        <color
+          rgba="0.64706 0.61961 0.58824 1" />
+      </material>
+    </visual>
+    <collision>
+      <origin
+        xyz="0 0 0"
+        rpy="0 0 0" />
+      <geometry>
+        <mesh
+          filename="package://KridtBot/meshes/diff_link.STL" />
+      </geometry>
+    </collision>
+  </link>
+  <joint
+    name="diff_jnt"
+    type="fixed">
+    <origin
+      xyz="-0.00062572 0.016887 -0.015618"
+      rpy="1.5708 0 -1.5708" />
+    <parent
+      link="base_link" />
+    <child
+      link="diff_link" />
+    <axis
+      xyz="0 0 0" />
+  </joint>
+  <link
+    name="left_diff_link">
+    <inertial>
+      <origin
+        xyz="-8.854E-07 -0.033684 -0.030541"
+        rpy="0 0 0" />
+      <mass
+        value="2.9663" />
+      <inertia
+        ixx="0.013273"
+        ixy="-3.2863E-08"
+        ixz="-4.8844E-08"
+        iyy="0.047575"
+        iyz="3.016E-08"
+        izz="0.05321" />
+    </inertial>
+    <visual>
+      <origin
+        xyz="0 0 0"
+        rpy="0 0 0" />
+      <geometry>
+        <mesh
+          filename="package://KridtBot/meshes/left_diff_link.STL" />
+      </geometry>
+      <material
+        name="">
+        <color
+          rgba="0.64706 0.61961 0.58824 1" />
+      </material>
+    </visual>
+    <collision>
+      <origin
+        xyz="0 0 0"
+        rpy="0 0 0" />
+      <geometry>
+        <mesh
+          filename="package://KridtBot/meshes/left_diff_link.STL" />
+      </geometry>
+    </collision>
+  </link>
+  <joint
+    name="left_diff_jnt"
+    type="revolute">
+    <origin
+      xyz="0 0 -0.28"
+      rpy="-3.1416 0 -3.1366" />
+    <parent
+      link="diff_link" />
+    <child
+      link="left_diff_link" />
+    <axis
+      xyz="0 0 1" />
+    <limit
+      lower="0"
+      upper="0"
+      effort="0"
+      velocity="0" />
+  </joint>
+  <link
+    name="left_rear_lin_link">
+    <inertial>
+      <origin
+        xyz="0.00095147 -0.0034915 0.19711"
+        rpy="0 0 0" />
+      <mass
+        value="0.44112" />
+      <inertia
+        ixx="0.00080168"
+        ixy="3.7318E-07"
+        ixz="-2.8679E-06"
+        iyy="0.00085013"
+        iyz="3.5668E-06"
+        izz="0.00022588" />
+    </inertial>
+    <visual>
+      <origin
+        xyz="0 0 0"
+        rpy="0 0 0" />
+      <geometry>
+        <mesh
+          filename="package://KridtBot/meshes/left_rear_lin_link.STL" />
+      </geometry>
+      <material
+        name="">
+        <color
+          rgba="0.62745 0.62745 0.62745 1" />
+      </material>
+    </visual>
+    <collision>
+      <origin
+        xyz="0 0 0"
+        rpy="0 0 0" />
+      <geometry>
+        <mesh
+          filename="package://KridtBot/meshes/left_rear_lin_link.STL" />
+      </geometry>
+    </collision>
+  </link>
+  <joint
+    name="left_rear_lin_jnt"
+    type="prismatic">
+    <origin
+      xyz="-0.216 -0.0010724 0"
+      rpy="-1.5708 0 0.0049647" />
+    <parent
+      link="left_diff_link" />
+    <child
+      link="left_rear_lin_link" />
+    <axis
+      xyz="0.0049647 0 0.99999" />
+    <limit
+      lower="0"
+      upper="0"
+      effort="0"
+      velocity="0" />
+  </joint>
+  <link
+    name="left_rear_rev_link">
+    <inertial>
+      <origin
+        xyz="-7.5958E-05 -0.0069814 0.060923"
+        rpy="0 0 0" />
+      <mass
+        value="1.3007" />
+      <inertia
+        ixx="0.0026916"
+        ixy="4.846E-07"
+        ixz="1.4471E-06"
+        iyy="0.0026895"
+        iyz="3.1405E-07"
+        izz="0.0046912" />
+    </inertial>
+    <visual>
+      <origin
+        xyz="0 0 0"
+        rpy="0 0 0" />
+      <geometry>
+        <mesh
+          filename="package://KridtBot/meshes/left_rear_rev_link.STL" />
+      </geometry>
+      <material
+        name="">
+        <color
+          rgba="0.25098 0.25098 0.25098 1" />
+      </material>
+    </visual>
+    <collision>
+      <origin
+        xyz="0 0 0"
+        rpy="0 0 0" />
+      <geometry>
+        <mesh
+          filename="package://KridtBot/meshes/left_rear_rev_link.STL" />
+      </geometry>
+    </collision>
+  </link>
+  <joint
+    name="left_rear_rev_jnt"
+    type="continuous">
+    <origin
+      xyz="0.0012505 0 0.25187"
+      rpy="1.5708 0 0" />
+    <parent
+      link="left_rear_lin_link" />
+    <child
+      link="left_rear_rev_link" />
+    <axis
+      xyz="0 0 1" />
+  </joint>
+  <link
+    name="front_left_lin_link">
+    <inertial>
+      <origin
+        xyz="0.00086415 -0.0034919 0.17949"
+        rpy="0 0 0" />
+      <mass
+        value="0.44112" />
+      <inertia
+        ixx="0.00080168"
+        ixy="3.8826E-07"
+        ixz="-2.8671E-06"
+        iyy="0.00085013"
+        iyz="3.5647E-06"
+        izz="0.00022588" />
+    </inertial>
+    <visual>
+      <origin
+        xyz="0 0 0"
+        rpy="0 0 0" />
+      <geometry>
+        <mesh
+          filename="package://KridtBot/meshes/front_left_lin_link.STL" />
+      </geometry>
+      <material
+        name="">
+        <color
+          rgba="0.62745 0.62745 0.62745 1" />
+      </material>
+    </visual>
+    <collision>
+      <origin
+        xyz="0 0 0"
+        rpy="0 0 0" />
+      <geometry>
+        <mesh
+          filename="package://KridtBot/meshes/front_left_lin_link.STL" />
+      </geometry>
+    </collision>
+  </link>
+  <joint
+    name="front_left_lin_jnt"
+    type="prismatic">
+    <origin
+      xyz="0.216 0.0010724 0"
+      rpy="-1.5708 0 0.0049647" />
+    <parent
+      link="left_diff_link" />
+    <child
+      link="front_left_lin_link" />
+    <axis
+      xyz="0.0049647 0 0.99999" />
+    <limit
+      lower="0"
+      upper="0"
+      effort="0"
+      velocity="0" />
+  </joint>
+  <link
+    name="left_front_rev_link">
+    <inertial>
+      <origin
+        xyz="-2.1691E-05 -0.0069321 0.060923"
+        rpy="0 0 0" />
+      <mass
+        value="1.3007" />
+      <inertia
+        ixx="0.0026896"
+        ixy="6.802E-07"
+        ixz="-4.5242E-07"
+        iyy="0.0026915"
+        iyz="-1.4099E-06"
+        izz="0.0046912" />
+    </inertial>
+    <visual>
+      <origin
+        xyz="0 0 0"
+        rpy="0 0 0" />
+      <geometry>
+        <mesh
+          filename="package://KridtBot/meshes/left_front_rev_link.STL" />
+      </geometry>
+      <material
+        name="">
+        <color
+          rgba="0.25098 0.25098 0.25098 1" />
+      </material>
+    </visual>
+    <collision>
+      <origin
+        xyz="0 0 0"
+        rpy="0 0 0" />
+      <geometry>
+        <mesh
+          filename="package://KridtBot/meshes/left_front_rev_link.STL" />
+      </geometry>
+    </collision>
+  </link>
+  <joint
+    name="left_front_rev_jnt"
+    type="continuous">
+    <origin
+      xyz="0.001163 0 0.23424"
+      rpy="1.5708 0 0" />
+    <parent
+      link="front_left_lin_link" />
+    <child
+      link="left_front_rev_link" />
+    <axis
+      xyz="0 0 1" />
+  </joint>
+  <link
+    name="rigth_diff_link">
+    <inertial>
+      <origin
+        xyz="6.4782E-05 -0.033689 -0.030541"
+        rpy="0 0 0" />
+      <mass
+        value="2.9663" />
+      <inertia
+        ixx="0.013273"
+        ixy="-7.293E-05"
+        ixz="-4.6692E-08"
+        iyy="0.047575"
+        iyz="-3.3395E-08"
+        izz="0.05321" />
+    </inertial>
+    <visual>
+      <origin
+        xyz="0 0 0"
+        rpy="0 0 0" />
+      <geometry>
+        <mesh
+          filename="package://KridtBot/meshes/rigth_diff_link.STL" />
+      </geometry>
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
Commit message: w

File: kridtbot/description/robot_core.xacro (robot description, xacro)
@@ -3,5 +3,5 @@
     <link
     name="base_link">
-    <inertial>
+    <!-- <inertial>
       <origin
         xyz="-0.00062572 0.0029573 -0.11694"
@@ -16,5 +16,5 @@
         iyz="-0.0045004"
         izz="0.19616" />
-    </inertial>
+    </inertial> -->
     <visual>
       <origin

Commit message: w

File: kridtbot/description/robot_core.xacro (robot description, xacro)
@@ -22,6 +22,7 @@
         rpy="0 0 0" />
       <geometry>
-        <mesh
-          filename="package://kridtbot/meshes/base_link.STL" />
+        <!-- <mesh
+          filename="package://kridtbot/meshes/base_link.STL" /> -->
+        <box size="0.5 0.5 0.5"/>
       </geometry>
       <material
@@ -36,6 +37,7 @@
         rpy="0 0 0" />
       <geometry>
-        <mesh
-          filename="package://kridtbot/meshes/base_link.STL" />
+        <!-- <mesh
+          filename="package://kridtbot/meshes/base_link.STL" /> -->
+        <box size="0.5 0.5 0.5"/>
       </geometry>
     </collision>

Commit message: w

File: kridtbot/description/robot_core.xacro (robot description, xacro)
@@ -22,7 +22,6 @@
         rpy="0 0 0" />
       <geometry>
-        <!-- <mesh
-          filename="package://kridtbot/meshes/base_link.STL" /> -->
-        <box size="0.5 0.5 0.5"/>
+        <mesh
+          filename="package://kridt-bot/kridtbot/meshes/base_link.STL" />
       </geometry>
       <material

Commit message: w

File: kridtbot/description/robot_core.xacro (robot description, xacro)
@@ -22,6 +22,5 @@
         rpy="0 0 0" />
       <geometry>
-        <mesh
-          filename="package://kridt-bot/kridtbot/meshes/base_link.STL" />
+        <mesh filename="file://$(robot_description)/meshes/base_link.STL"/>
       </geometry>
       <material

Commit message: w

File: kridtbot/description/robot_core.xacro (robot description, xacro)
@@ -22,5 +22,5 @@
         rpy="0 0 0" />
       <geometry>
-        <mesh filename="file://$(robot_description)/meshes/base_link.STL"/>
+        <mesh filename="file://kridtbot/meshes/base_link.STL"/>
       </geometry>
       <material

Commit message: w

File: kridtbot/description/robot_core.xacro (robot description, xacro)
@@ -22,5 +22,5 @@
         rpy="0 0 0" />
       <geometry>
-        <mesh filename="file://kridtbot/meshes/base_link.STL"/>
+        <mesh filename="package://kridtbot/meshes/base_link.STL" />
       </geometry>
       <material

Commit message: w

File: kridtbot/description/robot_core.xacro (robot description, xacro)
@@ -3,41 +3,4 @@
     <link
     name="base_link">
-    <!-- <inertial>
-      <origin
-        xyz="-0.00062572 0.0029573 -0.11694"
-        rpy="0 0 0" />
-      <mass
-        value="3.8611" />
-      <inertia
-        ixx="0.1509"
-        ixy="-3.2679E-16"
-        ixz="-3.3043E-17"
-        iyy="0.14248"
-        iyz="-0.0045004"
-        izz="0.19616" />
-    </inertial> -->
-    <visual>
-      <origin
-        xyz="0 0 0"
-        rpy="0 0 0" />
-      <geometry>
-        <mesh filename="package://kridtbot/meshes/base_link.STL" />
-      </geometry>
-      <material
-        name="">
-        <color
-          rgba="0.98824 0.73725 0.51765 1" />
-      </material>
-    </visual>
-    <collision>
-      <origin
-        xyz="0 0 0"
-        rpy="0 0 0" />
-      <geometry>
-        <!-- <mesh
-          filename="package://kridtbot/meshes/base_link.STL" /> -->
-        <box size="0.5 0.5 0.5"/>
-      </geometry>
-    </collision>
   </link>
   <link

Commit message: w

File: kridtbot/description/robot_core.xacro (robot description, xacro)
@@ -3,21 +3,4 @@
     <link
     name="base_link">
-  </link>
-  <link
-    name="diff_link">
-    <inertial>
-      <origin
-        xyz="6.3148E-06 0.0091271 1.2916E-05"
-        rpy="0 0 0" />
-      <mass
-        value="2.9137" />
-      <inertia
-        ixx="0.0037228"
-        ixy="5.5526E-08"
-        ixz="1.4073E-07"
-        iyy="0.0030992"
-        iyz="1.4623E-08"
-        izz="0.0022766" />
-    </inertial>
     <visual>
       <origin
@@ -25,397 +8,5 @@
         rpy="0 0 0" />
       <geometry>
-        <mesh
-          filename="package://kridtbot/meshes/diff_link.STL" />
-      </geometry>
-      <material
-        name="">
-        <color
-          rgba="0.64706 0.61961 0.58824 1" />
-      </material>
-    </visual>
-    <collision>
-      <origin
-        xyz="0 0 0"
-        rpy="0 0 0" />
-      <geometry>
-        <mesh
-          filename="package://KridtBot/meshes/diff_link.STL" />
-      </geometry>
-    </collision>
-  </link>
-  <joint
-    name="diff_jnt"
-    type="fixed">
-    <origin
-      xyz="-0.00062572 0.016887 -0.015618"
-      rpy="1.5708 0 -1.5708" />
-    <parent
-      link="base_link" />
-    <child
-      link="diff_link" />
-    <axis
-      xyz="0 0 0" />
-  </joint>
-  <link
-    name="left_diff_link">
-    <inertial>
-      <origin
-        xyz="-8.854E-07 -0.033684 -0.030541"
-        rpy="0 0 0" />
-      <mass
-        value="2.9663" />
-      <inertia
-        ixx="0.013273"
-        ixy="-3.2863E-08"
-        ixz="-4.8844E-08"
-        iyy="0.047575"
-        iyz="3.016E-08"
-        izz="0.05321" />
-    </inertial>
-    <visual>
-      <origin
-        xyz="0 0 0"
-        rpy="0 0 0" />
-      <geometry>
-        <mesh
-          filename="package://KridtBot/meshes/left_diff_link.STL" />
-      </geometry>
-      <material
-        name="">
-        <color
-          rgba="0.64706 0.61961 0.58824 1" />
-      </material>
-    </visual>
-    <collision>
-      <origin
-        xyz="0 0 0"
-        rpy="0 0 0" />
-      <geometry>
-        <mesh
-          filename="package://KridtBot/meshes/left_diff_link.STL" />
-      </geometry>
-    </collision>
-  </link>
-  <joint
-    name="left_diff_jnt"
-    type="revolute">
-    <origin
-      xyz="0 0 -0.28"
-      rpy="-3.1416 0 -3.1366" />
-    <parent
-      link="diff_link" />
-    <child
-      link="left_diff_link" />
-    <axis
-      xyz="0 0 1" />
-    <limit
-      lower="0"
-      upper="0"
-      effort="0"
-      velocity="0" />
-  </joint>
-  <link
-    name="left_rear_lin_link">
-    <inertial>
-      <origin
-        xyz="0.00095147 -0.0034915 0.19711"
-        rpy="0 0 0" />
-      <mass
-        value="0.44112" />
-      <inertia
-        ixx="0.00080168"
-        ixy="3.7318E-07"
-        ixz="-2.8679E-06"
-        iyy="0.00085013"
-        iyz="3.5668E-06"
-        izz="0.00022588" />
-    </inertial>
-    <visual>
-      <origin
-        xyz="0 0 0"
-        rpy="0 0 0" />
-      <geometry>
-        <mesh
-          filename="package://KridtBot/meshes/left_rear_lin_link.STL" />
-      </geometry>
-      <material
-        name="">
-        <color
-          rgba="0.62745 0.62745 0.62745 1" />
-      </material>
-    </visual>
-    <collision>
-      <origin
-        xyz="0 0 0"
-        rpy="0 0 0" />
-      <geometry>
-        <mesh
-          filename="package://KridtBot/meshes/left_rear_lin_link.STL" />
-      </geometry>
-    </collision>
-  </link>
-  <joint
-    name="left_rear_lin_jnt"
-    type="prismatic">
-    <origin
-      xyz="-0.216 -0.0010724 0"
-      rpy="-1.5708 0 0.0049647" />
-    <parent
-      link="left_diff_link" />
-    <child
-      link="left_rear_lin_link" />
-    <axis
-      xyz="0.0049647 0 0.99999" />
-    <limit
-      lower="0"
-      upper="0"
-      effort="0"
-      velocity="0" />
-  </joint>
-  <link
-    name="left_rear_rev_link">
-    <inertial>
-      <origin
-        xyz="-7.5958E-05 -0.0069814 0.060923"
-        rpy="0 0 0" />
-      <mass
-        value="1.3007" />
-      <inertia
-        ixx="0.0026916"
-        ixy="4.846E-07"
-        ixz="1.4471E-06"
-        iyy="0.0026895"
-        iyz="3.1405E-07"
-        izz="0.0046912" />
-    </inertial>
-    <visual>
-      <origin
-        xyz="0 0 0"
-        rpy="0 0 0" />
-      <geometry>
-        <mesh
-          filename="package://KridtBot/meshes/left_rear_rev_link.STL" />
-      </geometry>
-      <material
-        name="">
-        <color
-          rgba="0.25098 0.25098 0.25098 1" />
-      </material>
-    </visual>
-    <collision>
-      <origin
-        xyz="0 0 0"
-        rpy="0 0 0" />
-      <geometry>
-        <mesh
-          filename="package://KridtBot/meshes/left_rear_rev_link.STL" />
-      </geometry>
-    </collision>
-  </link>
-  <joint
-    name="left_rear_rev_jnt"
-    type="continuous">
-    <origin
-      xyz="0.0012505 0 0.25187"
-      rpy="1.5708 0 0" />
-    <parent
-      link="left_rear_lin_link" />
-    <child
-      link="left_rear_rev_link" />
-    <axis
-      xyz="0 0 1" />
-  </joint>
-  <link
-    name="front_left_lin_link">
-    <inertial>
-      <origin
-        xyz="0.00086415 -0.0034919 0.17949"
-        rpy="0 0 0" />
-      <mass
-        value="0.44112" />
-      <inertia
-        ixx="0.00080168"
-        ixy="3.8826E-07"
-        ixz="-2.8671E-06"
-        iyy="0.00085013"
-        iyz="3.5647E-06"
-        izz="0.00022588" />
-    </inertial>
-    <visual>
-      <origin
-        xyz="0 0 0"
-        rpy="0 0 0" />
-      <geometry>
-        <mesh
-          filename="package://KridtBot/meshes/front_left_lin_link.STL" />
-      </geometry>
-      <material
-        name="">
-        <color
-          rgba="0.62745 0.62745 0.62745 1" />
-      </material>
-    </visual>
-    <collision>
-      <origin
-        xyz="0 0 0"
-        rpy="0 0 0" />
-      <geometry>
-        <mesh
-          filename="package://KridtBot/meshes/front_left_lin_link.STL" />
-      </geometry>
-    </collision>
-  </link>
-  <joint
-    name="front_left_lin_jnt"
-    type="prismatic">
-    <origin
-      xyz="0.216 0.0010724 0"
-      rpy="-1.5708 0 0.0049647" />
-    <parent
-      link="left_diff_link" />
-    <child
-      link="front_left_lin_link" />
-    <axis
-      xyz="0.0049647 0 0.99999" />
-    <limit
-      lower="0"
-      upper="0"
-      effort="0"
-      velocity="0" />
-  </joint>
-  <link
-    name="left_front_rev_link">
-    <inertial>
-      <origin
-        xyz="-2.1691E-05 -0.0069321 0.060923"
-        rpy="0 0 0" />
-      <mass
-        value="1.3007" />
-      <inertia
-        ixx="0.0026896"
-        ixy="6.802E-07"
-        ixz="-4.5242E-07"
-        iyy="0.0026915"
-        iyz="-1.4099E-06"
-        izz="0.0046912" />
-    </inertial>
-    <visual>
-      <origin
-        xyz="0 0 0"
-        rpy="0 0 0" />
-      <geometry>
-        <mesh
-          filename="package://KridtBot/meshes/left_front_rev_link.STL" />
-      </geometry>
-      <material
-        name="">
-        <color
-          rgba="0.25098 0.25098 0.25098 1" />
-      </material>
-    </visual>
-    <collision>
-      <origin
-        xyz="0 0 0"
-        rpy="0 0 0" />
-      <geometry>
-        <mesh
-          filename="package://KridtBot/meshes/left_front_rev_link.STL" />
-      </geometry>
-    </collision>
-  </link>
-  <joint
-    name="left_front_rev_jnt"
-    type="continuous">
-    <origin
-      xyz="0.001163 0 0.23424"
-      rpy="1.5708 0 0" />
-    <parent
-      link="front_left_lin_link" />
-    <child
-      link="left_front_rev_link" />
-    <axis
-      xyz="0 0 1" />
-  </joint>
-  <link
-    name="rigth_diff_link">
-    <inertial>
-      <origin
-        xyz="6.4782E-05 -0.033689 -0.030541"
-        rpy="0 0 0" />
-      <mass
-        value="2.9663" />
-      <inertia
-        ixx="0.013273"
-        ixy="-7.293E-05"
-        ixz="-4.6692E-08"
-        iyy="0.047575"
-        iyz="-3.3395E-08"
-        izz="0.05321" />
-    </inertial>
-    <visual>
-      <origin
-        xyz="0 0 0"
-        rpy="0 0 0" />
-      <geometry>
-        <mesh
-          filename="package://KridtBot/meshes/rigth_diff_link.STL" />
-      </geometry>
-      <material
-        name="">
-        <color
-          rgba="0.64706 0.61961 0.58824 1" />
-      </material>
-    </visual>
-    <collision>
-      <origin
-        xyz="0 0 0"
-        rpy="0 0 0" />
-      <geometry>
-        <mesh
-          filename="package://KridtBot/meshes/rigth_diff_link.STL" />
-      </geometry>
-    </collision>
-  </link>
-  <joint
-    name="right_diff_jnt"
-    type="revolute">
-    <origin
-      xyz="0 0 0.28"
-      rpy="0 0 0" />
-    <parent
-      link="diff_link" />
-    <child
-      link="rigth_diff_link" />
-    <axis
-      xyz="0 0 1" />
-    <limit
-      lower="0"
-      upper="0"
-      effort="0"
-      velocity="0" />
-  </joint>
-  <link
-    name="right_rear_lin_link">
-    <inertial>
-      <origin
-        xyz="-0.00046851 -0.0035025 0.19574"
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
Commit message: f

File: kridtbot/description/robot_core.xacro (robot description, xacro)
@@ -8,5 +8,5 @@
         rpy="0 0 0" />
       <geometry>
-        <mesh filename="package://kridtbot/meshes/base_link.STL" />
+        <mesh filename="package://kridtbot/meshes/base_link.stl" />
       </geometry>
       <material

Commit message: w

File: kridtbot/description/robot_core.xacro (robot description, xacro)
@@ -8,5 +8,5 @@
         rpy="0 0 0" />
       <geometry>
-        <mesh filename="package://kridtbot/meshes/base_link.stl" />
+        <mesh filename="file://$(find kridtbot)/meshes/base_link.STL" />
       </geometry>
       <material

Commit message: w

File: kridtbot/description/robot_core.xacro (robot description, xacro)
@@ -8,5 +8,5 @@
         rpy="0 0 0" />
       <geometry>
-        <mesh filename="file://$(find kridtbot)/meshes/base_link.STL" />
+        <mesh filename="file://$(robot_description)/meshes/base_link.STL" />
       </geometry>
       <material

Commit message: w

File: kridtbot/description/robot_core.xacro (robot description, xacro)
@@ -8,5 +8,5 @@
         rpy="0 0 0" />
       <geometry>
-        <mesh filename="file://$(robot_description)/meshes/base_link.STL" />
+        <mesh filename="package://kridtbot/meshes/base_link.dae" />
       </geometry>
       <material
