Commit message: w

File: kridtbot/description/robot_core.xacro (robot description, xacro)
@@ -1,154 +1,34 @@
 <?xml version="1.0"?>
 <robot xmlns:xacro="http://www.ros.org/wiki/xacro">
-  <link
-    name="base_link">
-    <inertial>
-      <origin
-        xyz="-0.00062572 0.0029573 -0.11694"
-        rpy="0 0 0" />
-      <mass
-        value="3.8611" />
-      <inertia
-        ixx="0.1509"
-        ixy="-3.2679E-16"
-        ixz="-3.3043E-17"
-        iyy="0.14248"
-        iyz="-0.0045004"
-        izz="0.19616" />
-    </inertial>
+  <!-- BASE LINK-->
+  <link name="base_link">
+  </link>
+  <joint name="base_to_chassis" type="fixed">
+    <origin xyz="0 0 0" rpy="-3.1415 0 0"/>
+    <parent link="base_link"/>
+    <child link="chassis_link"/>
+  </joint>
+  <!-- CHASSIS LINK-->
+  <link name="chassis_link">
     <visual>
-      <origin
-        xyz="-0.00062572 0.0029573 -0.11694"
-        rpy="0 0 0" />
+      <origin xyz="0 0 0" rpy="0 0 0"/>
       <geometry>
-        <mesh
-          filename="file:$(find kridtbot)/meshes/base_link.STL" />
+        <mesh filename="file:$(find kridtbot)/meshes/base_link.STL"/>
       </geometry>
-      <material
-        name="">
-        <color
-          rgba="0.98824 0.73725 0.51765 1" />
-      </material>
     </visual>
-    <collision>
-      <origin
-        xyz="0 0 0"
-        rpy="0 0 0" />
+  </link>
+  <joint name="chassis_to_diff" type="fixed">
+    <origin xyz="-0.00062572 0.016893 -0.01406" rpy="1.5708 0 -1.5708"/>
+    <parent link="chassis_link"/>
+    <child link="diff_link"/>
+  </joint>
+  <!-- DIFF LINK-->
+  <link name="diff_link">
+    <visual>
+      <origin xyz="0 0 0" rpy="0 0 0"/>
       <geometry>
-        <mesh
-          filename="file:$(find kridtbot)/meshes/base_link.STL" />
+        <mesh filename="file:$(find kridtbot)/meshes/diff_link.STL"/>
       </geometry>
-    </collision>
+    </visual>
   </link>
-  <link
-    name="diff_link">
-    <inertial>
-      <origin
-        xyz="6.3148E-06 0.0091271 1.2916E-05"
-        rpy="0 0 0" />
-      <mass
-        value="2.9137" />
-      <inertia
-        ixx="0.0037228"
-        ixy="5.5526E-08"
-        ixz="1.4073E-07"
-        iyy="0.0030992"
-        iyz="1.4623E-08"
-        izz="0.0022766" />
-    </inertial>
-    <visual>
-      <origin
-      xyz="6.3148E-06 0.0091271 1.2916E-05"
-      rpy="0 0 0" />
-      <geometry>
-        <mesh
-          filename="file:$(find kridtbot)/meshes/diff_link.STL" />
-      </geometry>
-      <material
-        name="">
-        <color
-          rgba="0.64706 0.61961 0.58824 1" />
-      </material>
-    </visual>
-    <collision>
-      <origin
-        xyz="0 0 0"
-        rpy="0 0 0" />
-      <geometry>
-        <mesh
-          filename="file:$(find kridtbot)/meshes/diff_link.STL" />
-      </geometry>
-    </collision>
-  </link>
-  <joint
-    name="diff_jnt"
-    type="fixed">
-    <origin
-      xyz="-0.00062572 0.016887 -0.015618"
-      rpy="1.5708 0 -1.5708" />
-    <parent
-      link="base_link" />
-    <child
-      link="diff_link" />
-    <axis
-      xyz="0 0 0" />
-  </joint>
-  <link
-    name="left_diff_link">
-    <inertial>
-      <origin
-        xyz="-8.854E-07 -0.033684 -0.030541"
-        rpy="0 0 0" />
-      <mass
-        value="2.9663" />
-      <inertia
-        ixx="0.013273"
-        ixy="-3.2863E-08"
-        ixz="-4.8844E-08"
-        iyy="0.047575"
-        iyz="3.016E-08"
-        izz="0.05321" />
-    </inertial>
-    <visual>
-      <origin
-        xyz="-8.854E-07 -0.033684 -0.030541"
-        rpy="0 0 0" />
-      <geometry>
-        <mesh
-          filename="file:$(find kridtbot)/meshes/left_diff_link.STL" />
-      </geometry>
-      <material
-        name="">
-        <color
-          rgba="0.64706 0.61961 0.58824 1" />
-      </material>
-    </visual>
-    <collision>
-      <origin
-        xyz="0 0 0"
-        rpy="0 0 0" />
-      <geometry>
-        <mesh
-          filename="file:$(find kridtbot)/meshes/left_diff_link.STL" />
-      </geometry>
-    </collision>
-  </link>
-  <joint
-    name="left_diff_jnt"
-    type="revolute">
-    <origin
-      xyz="0 0 -0.28"
-      rpy="-3.1416 0 -3.1366" />
-    <parent
-      link="diff_link" />
-    <child
-      link="left_diff_link" />
-    <axis
-      xyz="0 0 1" />
-    <limit
-      lower="0"
-      upper="0"
-      effort="0"
-      velocity="0" />
-  </joint>
-  </robot>
+</robot>

Commit message: changes to urdf

File: kridtbot/description/robot_core.xacro (robot description, xacro)
@@ -32,3 +32,17 @@
     </visual>
   </link>
+  <joint name="diff_to_left_diff" type="revolute">
+    <origin xyz="0 0 -0.28" rpy="-3.1416 0 -3.1416"/>
+    <parent link="diff_link"/>
+    <child link="left_diff_link"/>
+  </joint>
+  <!-- _____________LEFT DIFF LINK____________-->
+  <link name="left_diff_link">
+    <visual>
+      <origin xyz="0 0 0" rpy="0 0 0"/>
+      <geometry>
+        <mesh filename="file:$(find kridtbot)/meshes/left_diff_link.STL"/>
+      </geometry>
+    </visual>
+  </link>
 </robot>

Commit message: Changes to urdf

File: kridtbot/description/robot_core.xacro (robot description, xacro)
@@ -34,4 +34,7 @@
   <joint name="diff_to_left_diff" type="revolute">
     <origin xyz="0 0 -0.28" rpy="-3.1416 0 -3.1416"/>
+    <limit>
+      effort="1000" lower="-1.5708" upper="1.5708" velocity="0.5"
+    </limit>
     <parent link="diff_link"/>
     <child link="left_diff_link"/>

Commit message: Changes to urdf

File: kridtbot/description/robot_core.xacro (robot description, xacro)
@@ -34,7 +34,6 @@
   <joint name="diff_to_left_diff" type="revolute">
     <origin xyz="0 0 -0.28" rpy="-3.1416 0 -3.1416"/>
-    <limit>
-      effort="1000" lower="-1.5708" upper="1.5708" velocity="0.5"
-    </limit>
+    <axis xyz="0 0 1"/>
+    <limit effort="1000" lower="-1.5708" upper="1.5708" velocity="0.5"/>
     <parent link="diff_link"/>
     <child link="left_diff_link"/>

Commit message: Changes to URDF

File: kridtbot/description/robot_core.xacro (robot description, xacro)
@@ -18,4 +18,5 @@
     </visual>
   </link>
+    <!-- _____________BASE TO CHASSIS JOINT____________-->
   <joint name="chassis_to_diff" type="fixed">
     <origin xyz="-0.00062572 0.016893 -0.01406" rpy="1.5708 0 -1.5708"/>
@@ -32,8 +33,7 @@
     </visual>
   </link>
+  <!-- _____________DIFF TO LEFT DIFF JOINT____________-->
   <joint name="diff_to_left_diff" type="revolute">
     <origin xyz="0 0 -0.28" rpy="-3.1416 0 -3.1416"/>
-    <axis xyz="0 0 1"/>
-    <limit effort="1000" lower="-1.5708" upper="1.5708" velocity="0.5"/>
     <parent link="diff_link"/>
     <child link="left_diff_link"/>
@@ -48,3 +48,23 @@
     </visual>
   </link>
+  <!-- _____________LEFT DIFF TO LEFT REAR LIN JOINT____________-->
+  <joint name="diff_to_left_diff" type="revolute">
+    <origin xyz="-0.216 -0.0010724 0" rpy="1.5708 0 0.0049647"/>
+    <parent link="diff_link"/>
+    <child link="left_diff_link"/>
+  </joint>
+  <!-- _____________LEFT REAR LIN LINK____________-->
+  <link name="left_diff_link">
+    <visual>
+      <origin xyz="0 0 0" rpy="0 0 0"/>
+      <geometry>
+        <mesh filename="file:$(find kridtbot)/meshes/left_diff_link.STL"/>
+      </geometry>
+    </visual>
+  </link>
+  <joint name="diff_to_left_diff" type="revolute">
+    <origin xyz="-0.216 -0.0010724 0" rpy="1.5708 0 0.0049647"/>
+    <parent link="diff_link"/>
+    <child link="left_diff_link"/>
+  </joint>
 </robot>

Commit message: changes to URDF

File: kridtbot/description/robot_core.xacro (robot description, xacro)
@@ -36,4 +36,6 @@
   <joint name="diff_to_left_diff" type="revolute">
     <origin xyz="0 0 -0.28" rpy="-3.1416 0 -3.1416"/>
+    <axis xyz="0 0 1"/>
+    <limit effort="1000" lower="-1.5708" upper="1.5708" velocity="10"/>
     <parent link="diff_link"/>
     <child link="left_diff_link"/>
@@ -49,22 +51,18 @@
   </link>
   <!-- _____________LEFT DIFF TO LEFT REAR LIN JOINT____________-->
-  <joint name="diff_to_left_diff" type="revolute">
+  <joint name="diff_to_left_diff" type="prismatic">
+    <limit effort="1000.0" lower="-0.3" upper="0" velocity="0.5"/>
     <origin xyz="-0.216 -0.0010724 0" rpy="1.5708 0 0.0049647"/>
-    <parent link="diff_link"/>
+    <parent link="left_diff_link"/>
     <child link="left_diff_link"/>
   </joint>
   <!-- _____________LEFT REAR LIN LINK____________-->
-  <link name="left_diff_link">
+  <link name="left_rear_lin_link">
     <visual>
       <origin xyz="0 0 0" rpy="0 0 0"/>
       <geometry>
-        <mesh filename="file:$(find kridtbot)/meshes/left_diff_link.STL"/>
+        <mesh filename="file:$(find kridtbot)/meshes/left_rear_lin_link.STL"/>
       </geometry>
     </visual>
   </link>
-  <joint name="diff_to_left_diff" type="revolute">
-    <origin xyz="-0.216 -0.0010724 0" rpy="1.5708 0 0.0049647"/>
-    <parent link="diff_link"/>
-    <child link="left_diff_link"/>
-  </joint>
 </robot>

Commit message: Changes to URDF

File: kridtbot/description/robot_core.xacro (robot description, xacro)
@@ -51,5 +51,5 @@
   </link>
   <!-- _____________LEFT DIFF TO LEFT REAR LIN JOINT____________-->
-  <joint name="diff_to_left_diff" type="prismatic">
+  <joint name="left_diff_to_left_rear_lin" type="prismatic">
     <limit effort="1000.0" lower="-0.3" upper="0" velocity="0.5"/>
     <origin xyz="-0.216 -0.0010724 0" rpy="1.5708 0 0.0049647"/>

Commit message: Changes to URDF

File: kridtbot/description/robot_core.xacro (robot description, xacro)
@@ -55,5 +55,5 @@
     <origin xyz="-0.216 -0.0010724 0" rpy="1.5708 0 0.0049647"/>
     <parent link="left_diff_link"/>
-    <child link="left_diff_link"/>
+    <child link="left_rear_lin_link"/>
   </joint>
   <!-- _____________LEFT REAR LIN LINK____________-->

Commit message: Changes to URDF

File: kridtbot/description/robot_core.xacro (robot description, xacro)
@@ -53,4 +53,5 @@
   <joint name="left_diff_to_left_rear_lin" type="prismatic">
     <limit effort="1000.0" lower="-0.3" upper="0" velocity="0.5"/>
+    <axis xyz="0 0 1"/>
     <origin xyz="-0.216 -0.0010724 0" rpy="1.5708 0 0.0049647"/>
     <parent link="left_diff_link"/>
@@ -66,3 +67,30 @@
     </visual>
   </link>
+<!-- _____________LEFT REAR REV LINK____________-->
+  <link name="left_rear_rev_link">
+    <visual>
+      <origin xyz="0 0 0" rpy="0 0 0"/>
+      <geometry>
+        <mesh filename="file:$(find kridtbot)/meshes/left_rear_rev_link.STL"/>
+      </geometry>
+    </visual>
+  </link>
+  <!-- _____________LEFT REAR LIN LINK____________-->
+  <link name="left_front_lin_link">
+    <visual>
+      <origin xyz="0 0 0" rpy="0 0 0"/>
+      <geometry>
+        <mesh filename="file:$(find kridtbot)/meshes/left_front_lin_link.STL"/>
+      </geometry>
+    </visual>
+  </link>
+<!-- _____________LEFT FRONT REV LINK____________-->
+  <link name="left_front_rev_link">
+    <visual>
+      <origin xyz="0 0 0" rpy="0 0 0"/>
+      <geometry>
+        <mesh filename="file:$(find kridtbot)/meshes/left_front_rev_link.STL"/>
+      </geometry>
+    </visual>
+  </link>
 </robot>

Commit message: Changes to URDF

File: kridtbot/description/robot_core.xacro (robot description, xacro)
@@ -52,7 +52,7 @@
   <!-- _____________LEFT DIFF TO LEFT REAR LIN JOINT____________-->
   <joint name="left_diff_to_left_rear_lin" type="prismatic">
-    <limit effort="1000.0" lower="-0.3" upper="0" velocity="0.5"/>
+    <limit effort="1000.0" lower="0" upper="0.13" velocity="0.5"/>
+    <origin xyz="-0.216 -0.0010724 0" rpy="-1.5708 0 0.0049647"/>
     <axis xyz="0 0 1"/>
-    <origin xyz="-0.216 -0.0010724 0" rpy="1.5708 0 0.0049647"/>
     <parent link="left_diff_link"/>
     <child link="left_rear_lin_link"/>
@@ -67,30 +67,3 @@
     </visual>
   </link>
-<!-- _____________LEFT REAR REV LINK____________-->
-  <link name="left_rear_rev_link">
-    <visual>
-      <origin xyz="0 0 0" rpy="0 0 0"/>
-      <geometry>
-        <mesh filename="file:$(find kridtbot)/meshes/left_rear_rev_link.STL"/>
-      </geometry>
-    </visual>
-  </link>
-  <!-- _____________LEFT REAR LIN LINK____________-->
-  <link name="left_front_lin_link">
-    <visual>
-      <origin xyz="0 0 0" rpy="0 0 0"/>
-      <geometry>
-        <mesh filename="file:$(find kridtbot)/meshes/left_front_lin_link.STL"/>
-      </geometry>
-    </visual>
-  </link>
-<!-- _____________LEFT FRONT REV LINK____________-->
-  <link name="left_front_rev_link">
-    <visual>
-      <origin xyz="0 0 0" rpy="0 0 0"/>
-      <geometry>
-        <mesh filename="file:$(find kridtbot)/meshes/left_front_rev_link.STL"/>
-      </geometry>
-    </visual>
-  </link>
 </robot>

Commit message: Changes to URDF

File: kridtbot/description/robot_core.xacro (robot description, xacro)
@@ -67,3 +67,52 @@
     </visual>
   </link>
+<!-- _____________LEFT REAR LIN TO LEFT REAR REV JOINT____________-->
+  <joint name="left_rear_lin_to_left_rear_rev" type="continuous">
+    <origin xyz="0.0012158 0 0.2449" rpy="1.5708 0 0"/>
+    <axis xyz="0 0 1"/>
+    <parent link="left_rear_lin_link"/>
+    <child link="left_rear_rev_link"/>
+  </joint>
+  <!-- _____________LEFT REAR REV LINK____________-->
+  <link name="left_rear_rev_link">
+    <visual>
+      <origin xyz="0 0 0" rpy="0 0 0"/>
+      <geometry>
+        <mesh filename="file:$(find kridtbot)/meshes/left_rear_rev_link.STL"/>
+      </geometry>
+    </visual>
+  </link>
+    <!-- _____________LEFT DIFF TO LEFT FRONT LIN JOINT____________-->
+  <joint name="left_diff_to_left_front_lin" type="prismatic">
+    <limit effort="1000.0" lower="0" upper="0.13" velocity="0.5"/>
+    <origin xyz="0.216 0.0010724 0" rpy="-1.5708 0 0.0049647"/>
+    <axis xyz="0 0 1"/>
+    <parent link="left_diff_link"/>
+    <child link="left_front_lin_link"/>
+  </joint>
+  <!-- _____________LEFT FRONT LIN LINK____________-->
+  <link name="left_front_lin_link">
+    <visual>
+      <origin xyz="0 0 0" rpy="0 0 0"/>
+      <geometry>
+        <mesh filename="file:$(find kridtbot)/meshes/left_front_lin_link.STL"/>
+      </geometry>
+    </visual>
+  </link>
+<!-- _____________LEFT FRONT LIN TO LEFT FRONT REV JOINT____________-->
+  <joint name="left_front_lin_to_left_front_rev" type="continuous">
+    <origin xyz="0.0012158 0 0.2449" rpy="1.5708 0 0"/>
+    <axis xyz="0 0 1"/>
+    <parent link="left_front_lin_link"/>
+    <child link="left_front_rev_link"/>
+  </joint>
+  <!-- _____________LEFT FRONT REV LINK____________-->
+  <link name="left_front_rev_link">
+    <visual>
+      <origin xyz="0 0 0" rpy="0 0 0"/>
+      <geometry>
+        <mesh filename="file:$(find kridtbot)/meshes/left_front_rev_link.STL"/>
+      </geometry>
+    </visual>
+  </link>
 </robot>

Commit message: Final changes to URDF

File: kridtbot/description/robot_core.xacro (robot description, xacro)
@@ -77,7 +77,7 @@
   <link name="left_rear_rev_link">
     <visual>
-      <origin xyz="0 0 0" rpy="0 0 0"/>
-      <geometry>
-        <mesh filename="file:$(find kridtbot)/meshes/left_rear_rev_link.STL"/>
+      <origin xyz="0 0 0.06266" rpy="0 0 0"/>
+      <geometry>
+        <cylinder radius="0.0865" length="0.05234"/>
       </geometry>
     </visual>
@@ -96,5 +96,5 @@
       <origin xyz="0 0 0" rpy="0 0 0"/>
       <geometry>
-        <mesh filename="file:$(find kridtbot)/meshes/left_front_lin_link.STL"/>
+        <mesh filename="file:$(find kridtbot)/meshes/front_left_lin_link.STL"/>
       </geometry>
     </visual>
@@ -110,9 +110,92 @@
   <link name="left_front_rev_link">
     <visual>
-      <origin xyz="0 0 0" rpy="0 0 0"/>
-      <geometry>
-        <mesh filename="file:$(find kridtbot)/meshes/left_front_rev_link.STL"/>
-      </geometry>
-    </visual>
-  </link>
+      <origin xyz="0 0 0.06266" rpy="0 0 0"/>
+      <geometry>
+        <cylinder radius="0.0865" length="0.05234"/>
+      </geometry>
+    </visual>
+  </link>
+    <!-- _____________DIFF TO RIGHT DIFF JOINT____________-->
+    <joint name="diff_to_right_diff" type="revolute">
+      <origin xyz="0 0 0.28" rpy="0 0 0"/>
+      <axis xyz="0 0 1"/>
+      <limit effort="1000" lower="-1.5708" upper="1.5708" velocity="10"/>
+      <parent link="diff_link"/>
+      <child link="right_diff_link"/>
+    </joint>
+    <!-- _____________RIGHT DIFF LINK____________-->
+    <link name="right_diff_link">
+      <visual>
+        <origin xyz="0 0 0" rpy="0 0 0"/>
+        <geometry>
+          <mesh filename="file:$(find kridtbot)/meshes/rigth_diff_link.STL"/>
+        </geometry>
+      </visual>
+    </link>
+    <!-- _____________RIGHT DIFF TO RIGHT REAR LIN JOINT____________-->
+    <joint name="right_diff_to_right_rear_lin" type="prismatic">
+      <limit effort="1000.0" lower="0" upper="0.13" velocity="0.5"/>
+      <origin xyz="-0.216 -0.0010724 0" rpy="-1.5708 0 0.0049647"/>
+      <axis xyz="0 0 1"/>
+      <parent link="right_diff_link"/>
+      <child link="right_rear_lin_link"/>
+    </joint>
+    <!-- _____________RIGHT REAR LIN LINK____________-->
+    <link name="right_rear_lin_link">
+      <visual>
+        <origin xyz="0 0 0" rpy="0 0 0"/>
+        <geometry>
+          <mesh filename="file:$(find kridtbot)/meshes/right_rear_lin_link.STL"/>
+        </geometry>
+      </visual>
+    </link>
+  <!-- _____________RIGHT REAR LIN TO RIGHT REAR REV JOINT____________-->
+    <joint name="right_rear_lin_to_right_rear_rev" type="continuous">
+      <origin xyz="0.0012158 0 0.2449" rpy="1.5708 0 0"/>
+      <axis xyz="0 0 1"/>
+      <parent link="right_rear_lin_link"/>
+      <child link="right_rear_rev_link"/>
+    </joint>
+    <!-- _____________RIGHT REAR REV LINK____________-->
+    <link name="right_rear_rev_link">
+      <visual>
+        <origin xyz="0 0 0.06266" rpy="0 0 0"/>
+        <geometry>
+          <cylinder radius="0.0865" length="0.05234"/>
+        </geometry>
+      </visual>
+    </link>
+      <!-- _____________RIGHT DIFF TO RIGHT FRONT LIN JOINT____________-->
+    <joint name="right_diff_to_right_front_lin" type="prismatic">
+      <limit effort="1000.0" lower="0" upper="0.13" velocity="0.5"/>
+      <origin xyz="0.216 0.0010724 0" rpy="-1.5708 0 0.0049647"/>
+      <axis xyz="0 0 1"/>
+      <parent link="right_diff_link"/>
+      <child link="right_front_lin_link"/>
+    </joint>
+    <!-- _____________RIGHT FRONT LIN LINK____________-->
+    <link name="right_front_lin_link">
+      <visual>
+        <origin xyz="0 0 0" rpy="0 0 0"/>
+        <geometry>
+          <mesh filename="file:$(find kridtbot)/meshes/right_front_lin_link.STL"/>
+        </geometry>
+      </visual>
+    </link>
+  <!-- _____________RIGHT FRONT LIN TO RIGHT FRONT REV JOINT____________-->
+    <joint name="right_front_lin_to_right_front_rev" type="continuous">
+      <origin xyz="0.0012158 0 0.2449" rpy="1.5708 0 0"/>
+      <axis xyz="0 0 1"/>
+      <parent link="right_front_lin_link"/>
+      <child link="right_front_rev_link"/>
+    </joint>
+    <!-- _____________RIGHT FRONT REV LINK____________-->
+    <link name="right_front_rev_link">
+      <visual>
+        <origin xyz="0 0 0.06266" rpy="0 0 0"/>
+        <geometry>
+          <cylinder radius="0.0865" length="0.05234"/>
+        </geometry>
+      </visual>
+    </link>
 </robot>

Commit message: Colors

File: kridtbot/description/robot_core.xacro (robot description, xacro)
@@ -1,4 +1,10 @@
 <?xml version="1.0"?>
 <robot xmlns:xacro="http://www.ros.org/wiki/xacro">
+<material name="orange">
+  <color rgba="${252/255} ${188/255} ${132/255} 1" />
+</materia>
+<material name="black">
+  <color rgba="${64/255} ${64/255} ${64/255} 1" />
+</materia>
   <!-- ________BASE LINK___________-->
   <link name="base_link">
@@ -16,4 +22,5 @@
         <mesh filename="file:$(find kridtbot)/meshes/base_link.STL"/>
       </geometry>
+      <material name = "orange"\>
     </visual>
   </link>
@@ -31,4 +38,5 @@
         <mesh filename="file:$(find kridtbot)/meshes/diff_link.STL"/>
       </geometry>
+      <material name = "black"\>
     </visual>
   </link>
@@ -48,4 +56,5 @@
         <mesh filename="file:$(find kridtbot)/meshes/left_diff_link.STL"/>
       </geometry>
+      <material name = "orange"\>
     </visual>
   </link>
@@ -65,4 +74,5 @@
         <mesh filename="file:$(find kridtbot)/meshes/left_rear_lin_link.STL"/>
       </geometry>
+      <material name = "black"\>
     </visual>
   </link>
@@ -81,4 +91,5 @@
         <cylinder radius="0.0865" length="0.05234"/>
       </geometry>
+      <material name = "black"\>
     </visual>
   </link>
@@ -98,4 +109,5 @@
         <mesh filename="file:$(find kridtbot)/meshes/front_left_lin_link.STL"/>
       </geometry>
+      <material name = "black"\>
     </visual>
   </link>
@@ -114,4 +126,5 @@
         <cylinder radius="0.0865" length="0.05234"/>
       </geometry>
+      <material name = "black"\>
     </visual>
   </link>
@@ -131,4 +144,5 @@
           <mesh filename="file:$(find kridtbot)/meshes/rigth_diff_link.STL"/>
         </geometry>
+        <material name = "orange"\>
       </visual>
     </link>
@@ -148,4 +162,5 @@
           <mesh filename="file:$(find kridtbot)/meshes/right_rear_lin_link.STL"/>
         </geometry>
+        <material name = "black"\>
       </visual>
     </link>
@@ -164,4 +179,5 @@
           <cylinder radius="0.0865" length="0.05234"/>
         </geometry>
+        <material name = "black"\>
       </visual>
     </link>
@@ -181,4 +197,5 @@
           <mesh filename="file:$(find kridtbot)/meshes/right_front_lin_link.STL"/>
         </geometry>
+        <material name = "black"\>
       </visual>
     </link>
@@ -197,4 +214,5 @@
           <cylinder radius="0.0865" length="0.05234"/>
         </geometry>
+        <material name = "black"\>
       </visual>
     </link>

Commit message: f

File: kridtbot/description/robot_core.xacro (robot description, xacro)
@@ -22,5 +22,5 @@
         <mesh filename="file:$(find kridtbot)/meshes/base_link.STL"/>
       </geometry>
-      <material name = "orange"\>
+      <material name="orange"\>
     </visual>
   </link>
