Commit message: h

File: kridtbot/description/robot_core.xacro (robot description, xacro)
@@ -3,8 +3,11 @@
 <material name="orange">
   <color rgba="${252/255} ${188/255} ${132/255} 1" />
-</materia>
+</material>
 <material name="black">
   <color rgba="${64/255} ${64/255} ${64/255} 1" />
-</materia>
+</material>
+<material name="mesh_color">
+  <color rgba="${0/255} ${0/255} ${255/255} 0.6" />
+</material>
   <!-- ________BASE LINK___________-->
   <link name="base_link">
@@ -22,6 +25,17 @@
         <mesh filename="file:$(find kridtbot)/meshes/base_link.STL"/>
       </geometry>
-      <material name="orange"\>
-    </visual>
+      <material name="orange"/>
+    </visual>
+    <collision>
+      <origin xyz="0 0 0" rpy="0 0 0"/>
+      <geometry>
+        <mesh filename="file:$(find kridtbot)/meshes/base_link.STL"/>
+      </geometry>
+      <material name="mesh_color"/>
+    </collision>
+    <inertial>
+      <mass value=""/>
+      <inertia ixx="" ixy="" ixz="" iyy="" iyz="" izz""/>
+    </inertial>
   </link>
     <!-- _____________BASE TO CHASSIS JOINT____________-->
@@ -38,5 +52,5 @@
         <mesh filename="file:$(find kridtbot)/meshes/diff_link.STL"/>
       </geometry>
-      <material name = "black"\>
+      <material name = "black"/>
     </visual>
   </link>
@@ -56,6 +70,13 @@
         <mesh filename="file:$(find kridtbot)/meshes/left_diff_link.STL"/>
       </geometry>
-      <material name = "orange"\>
-    </visual>
+      <material name = "black"/>
+    </visual>
+    <collision>
+      <origin xyz="0 0 0" rpy="0 0 0"/>
+      <geometry>
+        <mesh filename="file:$(find kridtbot)/meshes/left_diff_link.STL"/>
+      </geometry>
+      <material name="mesh_color"/>
+    </collision>
   </link>
   <!-- _____________LEFT DIFF TO LEFT REAR LIN JOINT____________-->
@@ -74,6 +95,13 @@
         <mesh filename="file:$(find kridtbot)/meshes/left_rear_lin_link.STL"/>
       </geometry>
-      <material name = "black"\>
-    </visual>
+      <material name = "black"/>
+    </visual>
+    <collision>
+      <origin xyz="0 0 0" rpy="0 0 0"/>
+      <geometry>
+        <mesh filename="file:$(find kridtbot)/meshes/left_rear_lin_link.STL"/>
+      </geometry>
+      <material name="mesh_color"/>
+    </collision>
   </link>
 <!-- _____________LEFT REAR LIN TO LEFT REAR REV JOINT____________-->
@@ -91,6 +119,13 @@
         <cylinder radius="0.0865" length="0.05234"/>
       </geometry>
-      <material name = "black"\>
-    </visual>
+      <material name = "orange"/>
+    </visual>
+    <collision>
+      <origin xyz="0 0 0.06266" rpy="0 0 0"/>
+      <geometry>
+        <cylinder radius="0.0865" length="0.05234"/>
+      </geometry>
+      <material name="mesh_color"/>
+    </collision>
   </link>
     <!-- _____________LEFT DIFF TO LEFT FRONT LIN JOINT____________-->
@@ -109,6 +144,13 @@
         <mesh filename="file:$(find kridtbot)/meshes/front_left_lin_link.STL"/>
       </geometry>
-      <material name = "black"\>
-    </visual>
+      <material name = "black"/>
+    </visual>
+    <collision>
+      <origin xyz="0 0 0" rpy="0 0 0"/>
+      <geometry>
+        <mesh filename="file:$(find kridtbot)/meshes/front_left_lin_link.STL"/>
+      </geometry>
+      <material name="mesh_color"/>
+    </collision>
   </link>
 <!-- _____________LEFT FRONT LIN TO LEFT FRONT REV JOINT____________-->
@@ -126,6 +168,13 @@
         <cylinder radius="0.0865" length="0.05234"/>
       </geometry>
-      <material name = "black"\>
-    </visual>
+      <material name = "orange"/>
+    </visual>
+    <collision>
+      <origin xyz="0 0 0.06266" rpy="0 0 0"/>
+      <geometry>
+        <cylinder radius="0.0865" length="0.05234"/>
+      </geometry>
+      <material name="mesh_color"/>
+    </collision>
   </link>
     <!-- _____________DIFF TO RIGHT DIFF JOINT____________-->
@@ -144,6 +193,13 @@
           <mesh filename="file:$(find kridtbot)/meshes/rigth_diff_link.STL"/>
         </geometry>
-        <material name = "orange"\>
-      </visual>
+        <material name = "black"/>
+      </visual>
+      <collision>
+        <origin xyz="0 0 0" rpy="0 0 0"/>
+        <geometry>
+          <mesh filename="file:$(find kridtbot)/meshes/rigth_diff_link.STL"/>
+        </geometry>
+        <material name="mesh_color"/>
+      </collision>
     </link>
     <!-- _____________RIGHT DIFF TO RIGHT REAR LIN JOINT____________-->
@@ -162,6 +218,13 @@
           <mesh filename="file:$(find kridtbot)/meshes/right_rear_lin_link.STL"/>
         </geometry>
-        <material name = "black"\>
-      </visual>
+        <material name = "black"/>
+      </visual>
+      <collision>
+        <origin xyz="0 0 0" rpy="0 0 0"/>
+        <geometry>
+          <mesh filename="file:$(find kridtbot)/meshes/right_rear_lin_link.STL"/>
+        </geometry>
+        <material name="mesh_color"/>
+      </collision>
     </link>
   <!-- _____________RIGHT REAR LIN TO RIGHT REAR REV JOINT____________-->
@@ -179,6 +242,13 @@
           <cylinder radius="0.0865" length="0.05234"/>
         </geometry>
-        <material name = "black"\>
-      </visual>
+        <material name = "orange"/>
+      </visual>
+      <collision>
+        <origin xyz="0 0 0.06266" rpy="0 0 0"/>
+        <geometry>
+          <cylinder radius="0.0865" length="0.05234"/>
+        </geometry>
+        <material name="mesh_color"/>
+      </collision>
     </link>
       <!-- _____________RIGHT DIFF TO RIGHT FRONT LIN JOINT____________-->
@@ -197,6 +267,13 @@
           <mesh filename="file:$(find kridtbot)/meshes/right_front_lin_link.STL"/>
         </geometry>
-        <material name = "black"\>
-      </visual>
+        <material name = "black"/>
+      </visual>
+      <collision>
+        <origin xyz="0 0 0" rpy="0 0 0"/>
+        <geometry>
+          <mesh filename="file:$(find kridtbot)/meshes/right_front_lin_link.STL"/>
+        </geometry>
+        <material name="mesh_color"/>
+      </collision>
     </link>
   <!-- _____________RIGHT FRONT LIN TO RIGHT FRONT REV JOINT____________-->
@@ -214,6 +291,13 @@
           <cylinder radius="0.0865" length="0.05234"/>
         </geometry>
-        <material name = "black"\>
-      </visual>
+        <material name = "orange"/>
+      </visual>
+      <collision>
+        <origin xyz="0 0 0.06266" rpy="0 0 0"/>
+        <geometry>
+          <cylinder radius="0.0865" length="0.05234"/>
+        </geometry>
+        <material name="mesh_color"/>
+      </collision>
     </link>
 </robot>

Commit message: h

File: kridtbot/description/robot_core.xacro (robot description, xacro)
@@ -35,6 +35,6 @@
     </collision>
     <inertial>
-      <mass value=""/>
-      <inertia ixx="" ixy="" ixz="" iyy="" iyz="" izz""/>
+      <mass value="11061"/>
+      <inertia ixx="" ixy="" ixz="" iyy="" iyz="" izz=""/>
     </inertial>
   </link>

Commit message: URDF inertia

File: kridtbot/description/robot_core.xacro (robot description, xacro)
@@ -35,6 +35,6 @@
     </collision>
     <inertial>
-      <mass value="11061"/>
-      <inertia ixx="" ixy="" ixz="" iyy="" iyz="" izz=""/>
+      <mass value="11.18100"/>
+      <inertia ixx="0.52" ixy=" 0.00" ixz="0.00" iyy="0.48" iyz=" 0.04" izz="0.60"/>
     </inertial>
   </link>
@@ -54,4 +54,8 @@
       <material name = "black"/>
     </visual>
+    <inertial>
+      <mass value="1.44"/>
+      <inertia ixx="2024193.31e-9" ixy="258.53e-9" ixz="-42.56e-9" iyy="1553917.67e-9" iyz=" 559.93e-9" izz="1298088.14e-9"/>
+    </inertial>
   </link>
   <!-- _____________DIFF TO LEFT DIFF JOINT____________-->
@@ -79,4 +83,8 @@
       <material name="mesh_color"/>
     </collision>
+    <inertial>
+      <mass value="7.30200"/>
+      <inertia ixx="133810302.00e-9" ixy="35430.13e-9" ixz="356.93e-9" iyy="282054578.10e-9" iyz="-2296.44e-9" izz="397598064.18e-9"/>
+    </inertial>
   </link>
   <!-- _____________LEFT DIFF TO LEFT REAR LIN JOINT____________-->
@@ -104,4 +112,8 @@
       <material name="mesh_color"/>
     </collision>
+    <inertial>
+      <mass value="1.04456"/>
+      <inertia ixx="59743728.97e-9" ixy="-5941.33e-9" ixz="293509.06e-9" iyy="59856745.28e-9" iyz=" -1015856.43e-9" izz="595093.96e-9"/>
+    </inertial>
   </link>
 <!-- _____________LEFT REAR LIN TO LEFT REAR REV JOINT____________-->
@@ -128,4 +140,8 @@
       <material name="mesh_color"/>
     </collision>
+    <inertial>
+      <mass value="1.01100"/>
+      <inertia ixx="5844491.97e-9" ixy="-376.28e-9" ixz="-3671.08e-9" iyy="5842839.83e-9" iyz="-796.72e-9" izz="3646247.90e-9"/>
+    </inertial>
   </link>
     <!-- _____________LEFT DIFF TO LEFT FRONT LIN JOINT____________-->
@@ -153,4 +169,8 @@
       <material name="mesh_color"/>
     </collision>
+    <inertial>
+      <mass value="1.04456"/>
+      <inertia ixx="59743728.97e-9" ixy="-5941.33e-9" ixz="293509.06e-9" iyy="59856745.28e-9" iyz=" -1015856.43e-9" izz="595093.96e-9"/>
+    </inertial>
   </link>
 <!-- _____________LEFT FRONT LIN TO LEFT FRONT REV JOINT____________-->
@@ -177,4 +197,8 @@
       <material name="mesh_color"/>
     </collision>
+    <inertial>
+      <mass value="1.01100"/>
+      <inertia ixx="5844491.97e-9" ixy="-376.28e-9" ixz="-3671.08e-9" iyy="5842839.83e-9" iyz="-796.72e-9" izz="3646247.90e-9"/>
+    </inertial>
   </link>
     <!-- _____________DIFF TO RIGHT DIFF JOINT____________-->
@@ -202,4 +226,8 @@
         <material name="mesh_color"/>
       </collision>
+    <inertial>
+      <mass value="7.30200"/>
+      <inertia ixx="133810688.94e-9" ixy="319399.82e-9" ixz="2255.98e-9" iyy="282053860.06e-9" iyz="-558.22e-9" izz="397597733.07e-9"/>
+    </inertial>
     </link>
     <!-- _____________RIGHT DIFF TO RIGHT REAR LIN JOINT____________-->
@@ -227,4 +255,8 @@
         <material name="mesh_color"/>
       </collision>
+    <inertial>
+      <mass value="1.04456"/>
+      <inertia ixx="59743728.97e-9" ixy="-5941.33e-9" ixz="293509.06e-9" iyy="59856745.28e-9" iyz=" -1015856.43e-9" izz="595093.96e-9"/>
+    </inertial>
     </link>
   <!-- _____________RIGHT REAR LIN TO RIGHT REAR REV JOINT____________-->
@@ -251,4 +283,8 @@
         <material name="mesh_color"/>
       </collision>
+    <inertial>
+      <mass value="1.01100"/>
+      <inertia ixx="5844491.97e-9" ixy="-376.28e-9" ixz="-3671.08e-9" iyy="5842839.83e-9" iyz="-796.72e-9" izz="3646247.90e-9"/>
+    </inertial>
     </link>
       <!-- _____________RIGHT DIFF TO RIGHT FRONT LIN JOINT____________-->
@@ -276,4 +312,8 @@
         <material name="mesh_color"/>
       </collision>
+    <inertial>
+      <mass value="1.04456"/>
+      <inertia ixx="59743728.97e-9" ixy="-5941.33e-9" ixz="293509.06e-9" iyy="59856745.28e-9" iyz=" -1015856.43e-9" izz="595093.96e-9"/>
+    </inertial>
     </link>
   <!-- _____________RIGHT FRONT LIN TO RIGHT FRONT REV JOINT____________-->
@@ -300,4 +340,8 @@
         <material name="mesh_color"/>
       </collision>
+    <inertial>
+      <mass value="1.01100"/>
+      <inertia ixx="5844491.97e-9" ixy="-376.28e-9" ixz="-3671.08e-9" iyy="5842839.83e-9" iyz="-796.72e-9" izz="3646247.90e-9"/>
+    </inertial>
     </link>
 </robot>

Commit message: w

File: kridtbot/description/robot_core.xacro (robot description, xacro)
@@ -38,4 +38,7 @@
       <inertia ixx="0.52" ixy=" 0.00" ixz="0.00" iyy="0.48" iyz=" 0.04" izz="0.60"/>
     </inertial>
+    <gazebo reference="chassis_link">
+      <material>Gazebo/Orange</material>
+    </gazebo>
   </link>
     <!-- _____________BASE TO CHASSIS JOINT____________-->

Commit message: w

File: kridtbot/description/robot_core.xacro (robot description, xacro)
@@ -61,4 +61,6 @@
       <inertia ixx="2024193.31e-9" ixy="258.53e-9" ixz="-42.56e-9" iyy="1553917.67e-9" iyz=" 559.93e-9" izz="1298088.14e-9"/>
     </inertial>
+    <gazebo reference="diff_link">
+    </gazebo>
   </link>
   <!-- _____________DIFF TO LEFT DIFF JOINT____________-->
@@ -90,4 +92,7 @@
       <inertia ixx="133810302.00e-9" ixy="35430.13e-9" ixz="356.93e-9" iyy="282054578.10e-9" iyz="-2296.44e-9" izz="397598064.18e-9"/>
     </inertial>
+    <gazebo reference="left_diff_link">
+      <material>Gazebo/Black</material>
+    </gazebo>
   </link>
   <!-- _____________LEFT DIFF TO LEFT REAR LIN JOINT____________-->
@@ -119,4 +124,7 @@
       <inertia ixx="59743728.97e-9" ixy="-5941.33e-9" ixz="293509.06e-9" iyy="59856745.28e-9" iyz=" -1015856.43e-9" izz="595093.96e-9"/>
     </inertial>
+    <gazebo reference="left_rear_lin_link">
+      <material>Gazebo/Black</material>
+    </gazebo>
   </link>
 <!-- _____________LEFT REAR LIN TO LEFT REAR REV JOINT____________-->
@@ -147,4 +155,7 @@
       <inertia ixx="5844491.97e-9" ixy="-376.28e-9" ixz="-3671.08e-9" iyy="5842839.83e-9" iyz="-796.72e-9" izz="3646247.90e-9"/>
     </inertial>
+    <gazebo reference="left_rear_rev_link">
+      <material>Gazebo/Orange</material>
+    </gazebo>
   </link>
     <!-- _____________LEFT DIFF TO LEFT FRONT LIN JOINT____________-->
@@ -176,4 +187,7 @@
       <inertia ixx="59743728.97e-9" ixy="-5941.33e-9" ixz="293509.06e-9" iyy="59856745.28e-9" iyz=" -1015856.43e-9" izz="595093.96e-9"/>
     </inertial>
+    <gazebo reference="left_front_lin_link">
+      <material>Gazebo/Black</material>
+    </gazebo>
   </link>
 <!-- _____________LEFT FRONT LIN TO LEFT FRONT REV JOINT____________-->
@@ -204,4 +218,7 @@
       <inertia ixx="5844491.97e-9" ixy="-376.28e-9" ixz="-3671.08e-9" iyy="5842839.83e-9" iyz="-796.72e-9" izz="3646247.90e-9"/>
     </inertial>
+    <gazebo reference="left_front_rev_link">
+      <material>Gazebo/Orange</material>
+    </gazebo>
   </link>
     <!-- _____________DIFF TO RIGHT DIFF JOINT____________-->
@@ -233,4 +250,7 @@
       <inertia ixx="133810688.94e-9" ixy="319399.82e-9" ixz="2255.98e-9" iyy="282053860.06e-9" iyz="-558.22e-9" izz="397597733.07e-9"/>
     </inertial>
+    <gazebo reference="right_diff_link">
+      <material>Gazebo/Black</material>
+    </gazebo>
     </link>
     <!-- _____________RIGHT DIFF TO RIGHT REAR LIN JOINT____________-->
@@ -262,4 +282,7 @@
       <inertia ixx="59743728.97e-9" ixy="-5941.33e-9" ixz="293509.06e-9" iyy="59856745.28e-9" iyz=" -1015856.43e-9" izz="595093.96e-9"/>
     </inertial>
+    <gazebo reference="right_rear_lin_link">
+      <material>Gazebo/Black</material>
+    </gazebo>
     </link>
   <!-- _____________RIGHT REAR LIN TO RIGHT REAR REV JOINT____________-->
@@ -290,4 +313,7 @@
       <inertia ixx="5844491.97e-9" ixy="-376.28e-9" ixz="-3671.08e-9" iyy="5842839.83e-9" iyz="-796.72e-9" izz="3646247.90e-9"/>
     </inertial>
+    <gazebo reference="right_rear_rev_link">
+      <material>Gazebo/Orange</material>
+    </gazebo>
     </link>
       <!-- _____________RIGHT DIFF TO RIGHT FRONT LIN JOINT____________-->
@@ -319,4 +345,7 @@
       <inertia ixx="59743728.97e-9" ixy="-5941.33e-9" ixz="293509.06e-9" iyy="59856745.28e-9" iyz=" -1015856.43e-9" izz="595093.96e-9"/>
     </inertial>
+    <gazebo reference="right_front_lin_link">
+      <material>Gazebo/Black</material>
+    </gazebo>
     </link>
   <!-- _____________RIGHT FRONT LIN TO RIGHT FRONT REV JOINT____________-->
@@ -347,4 +376,7 @@
       <inertia ixx="5844491.97e-9" ixy="-376.28e-9" ixz="-3671.08e-9" iyy="5842839.83e-9" iyz="-796.72e-9" izz="3646247.90e-9"/>
     </inertial>
+    <gazebo reference="right_front_rev_link">
+      <material>Gazebo/Orange</material>
+    </gazebo>
     </link>
 </robot>

Commit message: g

File: kridtbot/description/robot_core.xacro (robot description, xacro)
@@ -12,4 +12,5 @@
   <!-- ________BASE LINK___________-->
   <link name="base_link">
+    <origin xyz="0 0 0" rpy="0 0 0"/>
   </link>
   <joint name="base_to_chassis" type="fixed">

Commit message: g

File: kridtbot/description/robot_core.xacro (robot description, xacro)
@@ -72,5 +72,4 @@
     <parent link="diff_link"/>
     <child link="left_diff_link"/>
-    <mimic joint="diff_to_right_diff" multiplyer="-1.0"/>
   </joint>
   <!-- _____________LEFT DIFF LINK____________-->

Commit message: fd

File: kridtbot/description/robot_core.xacro (robot description, xacro)
@@ -10,5 +10,5 @@
   <color rgba="${0/255} ${0/255} ${255/255} 0.6" />
 </material>
-  <!-- ________BASE LINK___________-->
+  <!-- ________BASE LINK__________
   <link name="base_link">
     <origin xyz="0 0 0" rpy="0 0 0"/>
@@ -19,6 +19,7 @@
     <child link="chassis_link"/>
   </joint>
+_ -->
   <!-- _____________CHASSIS LINK_____________-->
-  <link name="chassis_link">
+  <link name="base_link">
     <visual>
       <origin xyz="0 0 0" rpy="0 0 0"/>
@@ -39,5 +40,5 @@
       <inertia ixx="0.52" ixy=" 0.00" ixz="0.00" iyy="0.48" iyz=" 0.04" izz="0.60"/>
     </inertial>
-    <gazebo reference="chassis_link">
+    <gazebo reference="base_link">
       <material>Gazebo/Orange</material>
     </gazebo>
@@ -46,5 +47,5 @@
   <joint name="chassis_to_diff" type="fixed">
     <origin xyz="-0.00062572 0.016893 -0.01406" rpy="1.5708 0 -1.5708"/>
-    <parent link="chassis_link"/>
+    <parent link="base_link"/>
     <child link="diff_link"/>
   </joint>

Commit message: f

File: kridtbot/description/robot_core.xacro (robot description, xacro)
@@ -10,5 +10,5 @@
   <color rgba="${0/255} ${0/255} ${255/255} 0.6" />
 </material>
-  <!-- ________BASE LINK__________
+  <!-- ________BASE LINK__________-->
   <link name="base_link">
     <origin xyz="0 0 0" rpy="0 0 0"/>
@@ -19,7 +19,6 @@
     <child link="chassis_link"/>
   </joint>
-_ -->
   <!-- _____________CHASSIS LINK_____________-->
-  <link name="base_link">
+  <link name="chassis_link">
     <visual>
       <origin xyz="0 0 0" rpy="0 0 0"/>
@@ -40,5 +39,5 @@
       <inertia ixx="0.52" ixy=" 0.00" ixz="0.00" iyy="0.48" iyz=" 0.04" izz="0.60"/>
     </inertial>
-    <gazebo reference="base_link">
+    <gazebo reference="chassis_link">
       <material>Gazebo/Orange</material>
     </gazebo>
@@ -47,5 +46,5 @@
   <joint name="chassis_to_diff" type="fixed">
     <origin xyz="-0.00062572 0.016893 -0.01406" rpy="1.5708 0 -1.5708"/>
-    <parent link="base_link"/>
+    <parent link="chassis_link"/>
     <child link="diff_link"/>
   </joint>

Commit message: d

File: kridtbot/description/robot_core.xacro (robot description, xacro)
@@ -12,5 +12,11 @@
   <!-- ________BASE LINK__________-->
   <link name="base_link">
+  </link>
+  <joint name="base_footprint_joint" type="fixed">
     <origin xyz="0 0 0" rpy="0 0 0"/>
+    <parent link="base_link"/>
+    <child link="base_footprint"/>
+  </joint>
+  <link name="base_footprint">
   </link>
   <joint name="base_to_chassis" type="fixed">

Commit message: f

File: kridtbot/description/robot_core.xacro (robot description, xacro)
@@ -45,8 +45,8 @@
       <inertia ixx="0.52" ixy=" 0.00" ixz="0.00" iyy="0.48" iyz=" 0.04" izz="0.60"/>
     </inertial>
-    <gazebo reference="chassis_link">
-      <material>Gazebo/Orange</material>
-    </gazebo>
-  </link>
+  </link>
+  <gazebo reference="chassis_link">
+    <material>Gazebo/Orange</material>
+  </gazebo>
     <!-- _____________BASE TO CHASSIS JOINT____________-->
   <joint name="chassis_to_diff" type="fixed">
@@ -64,11 +64,19 @@
       <material name = "black"/>
     </visual>
+    <collision>
+      <origin xyz="0 0 0" rpy="0 0 0"/>
+      <geometry>
+        <mesh filename="file:$(find kridtbot)/meshes/diff_link.STL"/>
+      </geometry>
+      <material name="mesh_color"/>
+    </collision>
     <inertial>
       <mass value="1.44"/>
       <inertia ixx="2024193.31e-9" ixy="258.53e-9" ixz="-42.56e-9" iyy="1553917.67e-9" iyz=" 559.93e-9" izz="1298088.14e-9"/>
     </inertial>
-    <gazebo reference="diff_link">
-    </gazebo>
-  </link>
+  </link>
+  <gazebo reference="diff_link">
+    <material>Gazebo/Orange</material>
+  </gazebo>
   <!-- _____________DIFF TO LEFT DIFF JOINT____________-->
   <joint name="diff_to_left_diff" type="revolute">
