Commit message: f

File: kridtbot/description/robot_core.xacro (robot description, xacro)
@@ -107,8 +107,8 @@
       <inertia ixx="133810302.00e-9" ixy="35430.13e-9" ixz="356.93e-9" iyy="282054578.10e-9" iyz="-2296.44e-9" izz="397598064.18e-9"/>
     </inertial>
-    <gazebo reference="left_diff_link">
-      <material>Gazebo/Black</material>
-    </gazebo>
-  </link>
+  </link>
+  <gazebo reference="left_diff_link">
+    <material>Gazebo/Black</material>
+  </gazebo>
   <!-- _____________LEFT DIFF TO LEFT REAR LIN JOINT____________-->
   <joint name="left_diff_to_left_rear_lin" type="prismatic">
@@ -139,8 +139,8 @@
       <inertia ixx="59743728.97e-9" ixy="-5941.33e-9" ixz="293509.06e-9" iyy="59856745.28e-9" iyz=" -1015856.43e-9" izz="595093.96e-9"/>
     </inertial>
-    <gazebo reference="left_rear_lin_link">
-      <material>Gazebo/Black</material>
-    </gazebo>
-  </link>
+  </link>
+  <gazebo reference="left_rear_lin_link">
+    <material>Gazebo/Black</material>
+  </gazebo>
 <!-- _____________LEFT REAR LIN TO LEFT REAR REV JOINT____________-->
   <joint name="left_rear_lin_to_left_rear_rev" type="continuous">
@@ -170,8 +170,8 @@
       <inertia ixx="5844491.97e-9" ixy="-376.28e-9" ixz="-3671.08e-9" iyy="5842839.83e-9" iyz="-796.72e-9" izz="3646247.90e-9"/>
     </inertial>
-    <gazebo reference="left_rear_rev_link">
-      <material>Gazebo/Orange</material>
-    </gazebo>
-  </link>
+  </link>
+  <gazebo reference="left_rear_rev_link">
+    <material>Gazebo/Orange</material>
+  </gazebo>
     <!-- _____________LEFT DIFF TO LEFT FRONT LIN JOINT____________-->
   <joint name="left_diff_to_left_front_lin" type="prismatic">
@@ -202,8 +202,8 @@
       <inertia ixx="59743728.97e-9" ixy="-5941.33e-9" ixz="293509.06e-9" iyy="59856745.28e-9" iyz=" -1015856.43e-9" izz="595093.96e-9"/>
     </inertial>
-    <gazebo reference="left_front_lin_link">
-      <material>Gazebo/Black</material>
-    </gazebo>
-  </link>
+  </link>
+  <gazebo reference="left_front_lin_link">
+    <material>Gazebo/Black</material>
+  </gazebo>
 <!-- _____________LEFT FRONT LIN TO LEFT FRONT REV JOINT____________-->
   <joint name="left_front_lin_to_left_front_rev" type="continuous">
@@ -265,8 +265,8 @@
       <inertia ixx="133810688.94e-9" ixy="319399.82e-9" ixz="2255.98e-9" iyy="282053860.06e-9" iyz="-558.22e-9" izz="397597733.07e-9"/>
     </inertial>
+    </link>
     <gazebo reference="right_diff_link">
       <material>Gazebo/Black</material>
     </gazebo>
-    </link>
     <!-- _____________RIGHT DIFF TO RIGHT REAR LIN JOINT____________-->
     <joint name="right_diff_to_right_rear_lin" type="prismatic">
@@ -297,8 +297,8 @@
       <inertia ixx="59743728.97e-9" ixy="-5941.33e-9" ixz="293509.06e-9" iyy="59856745.28e-9" iyz=" -1015856.43e-9" izz="595093.96e-9"/>
     </inertial>
+    </link>
     <gazebo reference="right_rear_lin_link">
       <material>Gazebo/Black</material>
     </gazebo>
-    </link>
   <!-- _____________RIGHT REAR LIN TO RIGHT REAR REV JOINT____________-->
     <joint name="right_rear_lin_to_right_rear_rev" type="continuous">
@@ -328,8 +328,8 @@
       <inertia ixx="5844491.97e-9" ixy="-376.28e-9" ixz="-3671.08e-9" iyy="5842839.83e-9" iyz="-796.72e-9" izz="3646247.90e-9"/>
     </inertial>
+    </link>
     <gazebo reference="right_rear_rev_link">
       <material>Gazebo/Orange</material>
     </gazebo>
-    </link>
       <!-- _____________RIGHT DIFF TO RIGHT FRONT LIN JOINT____________-->
     <joint name="right_diff_to_right_front_lin" type="prismatic">
@@ -360,8 +360,8 @@
       <inertia ixx="59743728.97e-9" ixy="-5941.33e-9" ixz="293509.06e-9" iyy="59856745.28e-9" iyz=" -1015856.43e-9" izz="595093.96e-9"/>
     </inertial>
+    </link>
     <gazebo reference="right_front_lin_link">
       <material>Gazebo/Black</material>
     </gazebo>
-    </link>
   <!-- _____________RIGHT FRONT LIN TO RIGHT FRONT REV JOINT____________-->
     <joint name="right_front_lin_to_right_front_rev" type="continuous">
@@ -391,7 +391,7 @@
       <inertia ixx="5844491.97e-9" ixy="-376.28e-9" ixz="-3671.08e-9" iyy="5842839.83e-9" iyz="-796.72e-9" izz="3646247.90e-9"/>
     </inertial>
+    </link>
     <gazebo reference="right_front_rev_link">
       <material>Gazebo/Orange</material>
     </gazebo>
-    </link>
 </robot>

Commit message: g

File: kridtbot/description/robot_core.xacro (robot description, xacro)
@@ -244,4 +244,5 @@
       <parent link="diff_link"/>
       <child link="right_diff_link"/>
+      <mimic joint="diff_to_left_diff" multiplier="-1"/>
     </joint>
     <!-- _____________RIGHT DIFF LINK____________-->

Commit message: f

File: kridtbot/description/robot_core.xacro (robot description, xacro)
@@ -48,4 +48,6 @@
   <gazebo reference="chassis_link">
     <material>Gazebo/Orange</material>
+    <mu1 value = "0.3"/>
+    <mu2 value = "0.3"/>
   </gazebo>
     <!-- _____________BASE TO CHASSIS JOINT____________-->
@@ -78,4 +80,6 @@
   <gazebo reference="diff_link">
     <material>Gazebo/Orange</material>
+    <mu1 value = "0.3"/>
+    <mu2 value = "0.3"/>
   </gazebo>
   <!-- _____________DIFF TO LEFT DIFF JOINT____________-->
@@ -110,4 +114,6 @@
   <gazebo reference="left_diff_link">
     <material>Gazebo/Black</material>
+    <mu1 value = "0.3"/>
+    <mu2 value = "0.3"/>
   </gazebo>
   <!-- _____________LEFT DIFF TO LEFT REAR LIN JOINT____________-->
@@ -244,5 +250,5 @@
       <parent link="diff_link"/>
       <child link="right_diff_link"/>
-      <mimic joint="diff_to_left_diff" multiplier="-1"/>
+      <mimic joint="diff_to_left_diff" multiplier="1"/>
     </joint>
     <!-- _____________RIGHT DIFF LINK____________-->
@@ -269,4 +275,6 @@
     <gazebo reference="right_diff_link">
       <material>Gazebo/Black</material>
+      <mu1 value = "0.3"/>
+      <mu2 value = "0.3"/>
     </gazebo>
     <!-- _____________RIGHT DIFF TO RIGHT REAR LIN JOINT____________-->

Commit message: f

File: kridtbot/description/robot_core.xacro (robot description, xacro)
@@ -83,5 +83,5 @@
   <link name="imu_link">
     <visual>
-      <origin xyz="0 0 0" rpy="0 0 0"/>
+      <origin xyz="-1.0 0 0" rpy="1.57079633 0 1.57079633"/>
       <geometry>
         <mesh filename="file:$(find kridtbot)/meshes/imu_link.STL"/>
@@ -90,5 +90,5 @@
     </visual>
     <collision>
-      <origin xyz="0 0 0" rpy="0 0 0"/>
+      <origin xyz="-1.0 0 0" rpy="1.57079633 0 1.57079633"/>
       <geometry>
         <mesh filename="file:$(find kridtbot)/meshes/imu_link.STL"/>

Commit message: Changes to urdf

File: kridtbot/description/robot_core.xacro (robot description, xacro)
@@ -64,5 +64,5 @@
         <mesh filename="file:$(find kridtbot)/meshes/diff_link.STL"/>
       </geometry>
-      <material name = "black"/>
+      <material name = "orange"/>
     </visual>
     <collision>
@@ -83,5 +83,5 @@
   <link name="imu_link">
     <visual>
-      <origin xyz="-1.0 0 0" rpy="1.57079633 0 1.57079633"/>
+      <origin xyz="-0.028 -0.019 -0.01" rpy="1.57079633 0 1.57079633"/>
       <geometry>
         <mesh filename="file:$(find kridtbot)/meshes/imu_link.STL"/>
@@ -90,5 +90,5 @@
     </visual>
     <collision>
-      <origin xyz="-1.0 0 0" rpy="1.57079633 0 1.57079633"/>
+      <origin xyz="0 0 0" rpy="0 0 0"/>
       <geometry>
         <mesh filename="file:$(find kridtbot)/meshes/imu_link.STL"/>
@@ -101,10 +101,7 @@
     </inertial>
   </link>
-  <gazebo reference="imu_link">
-    <material>Gazebo/Orange</material>
-  </gazebo>
   <!-- _____________DIFF TO IMU JOINT____________-->
   <joint name="diff_to_imu" type="fixed">
-    <origin xyz="-1.0 0 0" rpy="1.57079633 0 1.57079633"/>
+    <origin xyz="0 -0.038 0" rpy="1.57079633 3.14159265 0"/>
     <parent link="diff_link"/>
     <child link="imu_link"/>
